Commit message: Fix mh50 flange joint
Co-authored-by: Claude <no-reply@anthropic.com>

File: motoman_mh50_support/urdf/mh50_macro.xacro (robot description, xacro)
@@ -149,5 +149,5 @@
     <!-- ROS-Industrial 'flange' frame, attachment point for EEF models -->
     <link name="${prefix}flange"/>
-    <joint name="${prefix}link_6_t-flange" type="fixed">
+    <joint name="${prefix}joint_6_t-flange" type="fixed">
       <origin xyz="0.175 0 0" rpy="0 0 0"/>
       <parent link="${prefix}link_6_t"/>

Commit message: feat: Change link and joint names (#2)
* Reconcile link/joint names to S/L/U/R/B/T convention

---------

Co-authored-by: Claude <no-reply@anthropic.com>

File: motoman_mh50_support/urdf/mh50_macro.xacro (robot description, xacro)
@@ -17,5 +17,5 @@
         </collision>
     </link>
-    <link name="${prefix}link_1">
+    <link name="${prefix}link_1_s">
         <visual>
             <geometry>
@@ -30,5 +30,5 @@
         </collision>
     </link>
-    <link name="${prefix}link_2">
+    <link name="${prefix}link_2_l">
         <visual>
             <geometry>
@@ -43,5 +43,5 @@
         </collision>
     </link>
-    <link name="${prefix}link_3">
+    <link name="${prefix}link_3_u">
         <visual>
             <geometry>
@@ -56,5 +56,5 @@
         </collision>
     </link>
-    <link name="${prefix}link_4">
+    <link name="${prefix}link_4_r">
         <visual>
             <geometry>
@@ -69,5 +69,5 @@
         </collision>
     </link>
-    <link name="${prefix}link_5">
+    <link name="${prefix}link_5_b">
         <visual>
             <geometry>
@@ -82,5 +82,5 @@
         </collision>
     </link>
-    <link name="${prefix}link_6">
+    <link name="${prefix}link_6_t">
         <visual>
             <geometry>
@@ -97,42 +97,42 @@
     <!-- end of link list -->
     <!-- joint list -->
-    <joint name="${prefix}joint_1" type="revolute">
+    <joint name="${prefix}joint_1_s" type="revolute">
         <parent link="${prefix}base_link"/>
-        <child link="${prefix}link_1"/>
+        <child link="${prefix}link_1_s"/>
         <origin xyz="0 0 0.540" rpy="0 0 0" />
         <axis xyz="0 0 1" />
         <limit lower="${radians(-180)}" upper="${radians(180)}" effort="4903.32" velocity="${radians(180)}"/>
     </joint>
-    <joint name="${prefix}joint_2" type="revolute">
-        <parent link="${prefix}link_1"/>
-        <child link="${prefix}link_2"/>
+    <joint name="${prefix}joint_2_l" type="revolute">
+        <parent link="${prefix}link_1_s"/>
+        <child link="${prefix}link_2_l"/>
         <origin xyz="0.145 0 0" rpy="0 0 0" />
         <axis xyz="0 1 0" />
         <limit lower="${radians(-90)}" upper="${radians(135)}" effort="6276.26" velocity="${radians(178)}"/>
     </joint>
-    <joint name="${prefix}joint_3" type="revolute">
-        <parent link="${prefix}link_2"/>
-        <child link="${prefix}link_3"/>
+    <joint name="${prefix}joint_3_u" type="revolute">
+        <parent link="${prefix}link_2_l"/>
+        <child link="${prefix}link_3_u"/>
         <origin xyz="0 0 0.870" rpy="0 0 0" />
         <axis xyz="0 -1 0" />
         <limit lower="${radians(-80)}" upper="${radians(206)}" effort="2745.86" velocity="${radians(178)}"/>
     </joint>
-    <joint name="${prefix}joint_4" type="revolute">
-        <parent link="${prefix}link_3"/>
-        <child link="${prefix}link_4"/>
+    <joint name="${prefix}joint_4_r" type="revolute">
+        <parent link="${prefix}link_3_u"/>
+        <child link="${prefix}link_4_r"/>
         <origin xyz="1.025 0 0.210" rpy="0 0 0"/>
         <axis xyz="-1 0 0" />
         <limit lower="${radians(-360)}" upper="${radians(360)}" effort="823.76" velocity="${radians(250)}"/>
     </joint>
-    <joint name="${prefix}joint_5" type="revolute">
-        <parent link="${prefix}link_4"/>
-        <child link="${prefix}link_5"/>
+    <joint name="${prefix}joint_5_b" type="revolute">
+        <parent link="${prefix}link_4_r"/>
+        <child link="${prefix}link_5_b"/>
         <origin xyz="0 0 0" rpy="0 0 0" />
         <axis xyz="0 -1 0" />
         <limit lower="${radians(-125)}" upper="${radians(125)}" effort="706.08" velocity="${radians(250)}"/>
     </joint>
-    <joint name="${prefix}joint_6" type="revolute">
-        <parent link="${prefix}link_5"/>
-        <child link="${prefix}link_6"/>
+    <joint name="${prefix}joint_6_t" type="revolute">
+        <parent link="${prefix}link_5_b"/>
+        <child link="${prefix}link_6_t"/>
         <origin xyz="0 0 0" rpy="0 0 0" />
         <axis xyz="-1 0 0" />
@@ -149,7 +149,7 @@
     <!-- ROS-Industrial 'flange' frame, attachment point for EEF models -->
     <link name="${prefix}flange"/>
-    <joint name="${prefix}joint_6-flange" type="fixed">
+    <joint name="${prefix}joint_6_t-flange" type="fixed">
       <origin xyz="0.175 0 0" rpy="0 0 0"/>
-      <parent link="${prefix}link_6"/>
+      <parent link="${prefix}link_6_t"/>
       <child link="${prefix}flange"/>
     </joint>
