Commit message: Add kinematic offset capability to d500, mh1655, ar2010, gp20hl, and gp180

File: motoman_ar2010_support/urdf/ar2010.xacro (robot description, xacro)
@@ -2,4 +2,5 @@
 <robot name="motoman_ar2010" xmlns:xacro="http://ros.org/wiki/xacro">
   <xacro:include filename="$(find motoman_ar2010_support)/urdf/ar2010_macro.xacro" />
-  <xacro:motoman_ar2010 prefix=""/>
+  <xacro:property name="kinematics_offsets" value="${xacro.load_yaml('$(find motoman_ar2010_support)' + '/config/default_kinematic_offsets.yaml')}"/>
+  <xacro:motoman_ar2010 prefix="" kinematic_offsets="${kinematics_offsets['kinematic_offsets']}"/>
 </robot>

File: motoman_ar2010_support/urdf/ar2010_macro.xacro (robot description, xacro)
@@ -1,5 +1,5 @@
 <?xml version="1.0" ?>
 <robot xmlns:xacro="http://ros.org/wiki/xacro">
-  <xacro:macro name="motoman_ar2010" params="prefix">
+  <xacro:macro name="motoman_ar2010" params="prefix kinematic_offsets">
     <xacro:include filename="$(find motoman_resources)/urdf/common_materials.xacro"/>
     <!-- link list -->
@@ -101,5 +101,5 @@
       <parent link="${prefix}base_link"/>
       <child link="${prefix}link_1_s"/>
-      <origin xyz="0 0 0.505" rpy="0 0 0"/>
+      <origin xyz="${0 + kinematic_offsets['1_s']['x']} ${0 + kinematic_offsets['1_s']['y']} ${0.505 + kinematic_offsets['1_s']['z']}" rpy="${0 + kinematic_offsets['1_s']['roll']} ${0 + kinematic_offsets['1_s']['pitch']} ${0 + kinematic_offsets['1_s']['yaw']}"/>
       <axis xyz="0 0 1"/>
       <limit lower="${radians(-180)}" upper="${radians(180)}" effort="3087" velocity="${radians(210)}"/>
@@ -108,5 +108,5 @@
       <parent link="${prefix}link_1_s"/>
       <child link="${prefix}link_2_l"/>
-      <origin xyz="0.150 0 0" rpy="${radians(90)} ${radians(-90)} ${radians(-180)}"/>
+      <origin xyz="${0.150 + kinematic_offsets['2_l']['x']} ${0 + kinematic_offsets['2_l']['y']} ${0 + kinematic_offsets['2_l']['z']}" rpy="${radians(90) + kinematic_offsets['2_l']['roll']} ${radians(-90) + kinematic_offsets['2_l']['pitch']} ${radians(-180) + kinematic_offsets['2_l']['yaw']}"/>
       <axis xyz="0 0 1"/>
       <limit lower="${radians(-105)}" upper="${radians(155)}" effort="3087" velocity="${radians(210)}"/>
@@ -115,5 +115,5 @@
       <parent link="${prefix}link_2_l"/>
       <child link="${prefix}link_3_u"/>
-      <origin xyz="0.760 0 0" rpy="${radians(180)} 0 0"/>
+      <origin xyz="${0.760 + kinematic_offsets['3_u']['x']} ${0 + kinematic_offsets['3_u']['y']} ${0 + kinematic_offsets['3_u']['z']}" rpy="${radians(180) + kinematic_offsets['3_u']['roll']} ${0 + kinematic_offsets['3_u']['pitch']} ${0 + kinematic_offsets['3_u']['yaw']}"/>
       <axis xyz="0 0 1"/>
       <limit lower="${radians(-86)}" upper="${radians(160)}" effort="926.1" velocity="${radians(220)}"/>
@@ -122,5 +122,5 @@
       <parent link="${prefix}link_3_u"/>
       <child link="${prefix}link_4_r"/>
-      <origin xyz="0.200 -1.082 0" rpy="${radians(-90)} 0 0"/>
+      <origin xyz="${0.200 + kinematic_offsets['4_r']['x']} ${-1.082 + kinematic_offsets['4_r']['y']} ${0 + kinematic_offsets['4_r']['z']}" rpy="${radians(-90) + kinematic_offsets['4_r']['roll']} ${0 + kinematic_offsets['4_r']['pitch']} ${0 + kinematic_offsets['4_r']['yaw']}"/>
       <axis xyz="0 0 1"/>
       <limit lower="${radians(-200)}" upper="${radians(200)}" effort="78.4" velocity="${radians(435)}"/>
@@ -129,5 +129,5 @@
       <parent link="${prefix}link_4_r"/>
       <child link="${prefix}link_5_b"/>
-      <origin xyz="0 0 0" rpy="${radians(90)} 0 0"/>
+      <origin xyz="${0 + kinematic_offsets['5_b']['x']} ${0 + kinematic_offsets['5_b']['y']} ${0 + kinematic_offsets['5_b']['z']}" rpy="${radians(90) + kinematic_offsets['5_b']['roll']} ${0 + kinematic_offsets['5_b']['pitch']} ${0 + kinematic_offsets['5_b']['yaw']}"/>
       <axis xyz="0 0 1"/>
       <limit lower="${radians(-150)}" upper="${radians(150)}" effort="67.03" velocity="${radians(435)}"/>
@@ -136,5 +136,5 @@
       <parent link="${prefix}link_5_b"/>
       <child link="${prefix}link_6_t"/>
-      <origin xyz="0 -0.100 0" rpy="${radians(-90)} 0 0"/>
+      <origin xyz="${0 + kinematic_offsets['6_t']['x']} ${-0.100 + kinematic_offsets['6_t']['y']} ${0 + kinematic_offsets['6_t']['z']}" rpy="${radians(-90) + kinematic_offsets['6_t']['roll']} ${0 + kinematic_offsets['6_t']['pitch']} ${0 + kinematic_offsets['6_t']['yaw']}"/>
       <axis xyz="0 0 1"/>
       <limit lower="${radians(-455)}" upper="${radians(455)}" effort="33.3" velocity="${radians(700)}"/>

File: motoman_gp180_support/urdf/gp180.xacro (robot description, xacro)
@@ -2,4 +2,5 @@
 <robot name="motoman_gp180" xmlns:xacro="http://ros.org/wiki/xacro">
     <xacro:include filename="$(find motoman_gp180_support)/urdf/gp180_macro.xacro" />
-    <xacro:motoman_gp180 prefix=""/>
+  <xacro:property name="kinematics_offsets" value="${xacro.load_yaml('$(find motoman_gp180_support)' + '/config/default_kinematic_offsets.yaml')}"/>
+    <xacro:motoman_gp180 prefix="" kinematic_offsets="${kinematics_offsets['kinematic_offsets']}"/>
 </robot>

File: motoman_gp180_support/urdf/gp180_macro.xacro (robot description, xacro)
@@ -1,5 +1,5 @@
 <?xml version="1.0" ?>
 <robot xmlns:xacro="http://ros.org/wiki/xacro">
-<xacro:macro name="motoman_gp180" params="prefix">
+<xacro:macro name="motoman_gp180" params="prefix kinematic_offsets">
     <xacro:include filename="$(find motoman_resources)/urdf/common_materials.xacro"/>
     <!-- link list -->
@@ -110,5 +110,5 @@
         <parent link="${prefix}base_link"/>
         <child link="${prefix}link_1_s"/>
-        <origin xyz="0 0 0.650" rpy="0 0 0" />
+        <origin xyz="${0 + kinematic_offsets['1_s']['x']} ${0 + kinematic_offsets['1_s']['y']} ${0.650 + kinematic_offsets['1_s']['z']}" rpy="${0 + kinematic_offsets['1_s']['roll']} ${0 + kinematic_offsets['1_s']['pitch']} ${0 + kinematic_offsets['1_s']['yaw']}" />
         <axis xyz="0 0 1" />
         <limit lower="${radians(-180)}" upper="${radians(180)}" effort="8237.59" velocity="${radians(125)}"/>
@@ -117,5 +117,5 @@
         <parent link="${prefix}link_1_s"/>
         <child link="${prefix}link_2_l"/>
-        <origin xyz="0.325 0 0" rpy="0 ${radians(-90)} ${radians(-90)}" />
+        <origin xyz="${0.325 + kinematic_offsets['2_l']['x']} ${0 + kinematic_offsets['2_l']['y']} ${0 + kinematic_offsets['2_l']['z']}" rpy="${0 + kinematic_offsets['2_l']['roll']} ${radians(-90) + kinematic_offsets['2_l']['pitch']} ${radians(-90) + kinematic_offsets['2_l']['yaw']}" />
         <axis xyz="0 0 1" />
         <limit lower="${radians(-60)}" upper="${radians(76)}" effort="10419.57" velocity="${radians(115)}"/>
@@ -124,5 +124,5 @@
         <parent link="${prefix}link_2_l"/>
         <child link="${prefix}link_3_u"/>
-        <origin xyz="1.150 0 0" rpy="${radians(180)} 0 0" />
+        <origin xyz="${1.150 + kinematic_offsets['3_u']['x']} ${0 + kinematic_offsets['3_u']['y']} ${0 + kinematic_offsets['3_u']['z']}" rpy="${radians(180) + kinematic_offsets['3_u']['roll']} ${0 + kinematic_offsets['3_u']['pitch']} ${0 + kinematic_offsets['3_u']['yaw']}" />
         <axis xyz="0 0 1" />
         <limit lower="${radians(-86)}" upper="${radians(90)}" effort="7453.05" velocity="${radians(125)}"/>
@@ -131,5 +131,5 @@
         <parent link="${prefix}link_3_u"/>
         <child link="${prefix}link_4_r"/>
-        <origin xyz="0.300 -1.225 0" rpy="${radians(-90)} 0 0" />
+        <origin xyz="${0.300 + kinematic_offsets['4_r']['x']} ${-1.225 + kinematic_offsets['4_r']['y']} ${0 + kinematic_offsets['4_r']['z']}" rpy="${radians(-90) + kinematic_offsets['4_r']['roll']} ${0 + kinematic_offsets['4_r']['pitch']} ${0 + kinematic_offsets['4_r']['yaw']}" />
         <axis xyz="0 0 1" />
         <limit lower="${radians(-360)}" upper="${radians(360)}" effort="1671.05" velocity="${radians(182)}"/>
@@ -138,5 +138,5 @@
         <parent link="${prefix}link_4_r"/>
         <child link="${prefix}link_5_b"/>
-        <origin xyz="0 0 0" rpy="${radians(90)} 0 0" />
+        <origin xyz="${0 + kinematic_offsets['5_b']['x']} ${0 + kinematic_offsets['5_b']['y']} ${0 + kinematic_offsets['5_b']['z']}" rpy="${radians(90) + kinematic_offsets['5_b']['roll']} ${0 + kinematic_offsets['5_b']['pitch']} ${0 + kinematic_offsets['5_b']['yaw']}" />
         <axis xyz="0 0 1" />
         <limit lower="${radians(-130)}" upper="${radians(130)}" effort="1081.18" velocity="${radians(175)}"/>
@@ -145,5 +145,5 @@
         <parent link="${prefix}link_5_b"/>
         <child link="${prefix}link_6_t"/>
-        <origin xyz="0 -0.225 0" rpy="${radians(-90)} 0 0" />
+        <origin xyz="${0 + kinematic_offsets['6_t']['x']} ${-0.225 + kinematic_offsets['6_t']['y']} ${0 + kinematic_offsets['6_t']['z']}" rpy="${radians(-90) + kinematic_offsets['6_t']['roll']} ${0 + kinematic_offsets['6_t']['pitch']} ${0 + kinematic_offsets['6_t']['yaw']}" />
         <axis xyz="0 0 1" />
         <limit lower="${radians(-360)}" upper="${radians(360)}" effort="926.73" velocity="${radians(265)}"/>

File: motoman_gp20hl_support/urdf/gp20hl.xacro (robot description, xacro)
@@ -2,4 +2,5 @@
 <robot name="motoman_gp20hl" xmlns:xacro="http://ros.org/wiki/xacro">
   <xacro:include filename="$(find motoman_gp20hl_support)/urdf/gp20hl_macro.xacro" />
-  <xacro:motoman_gp20hl prefix=""/>
+  <xacro:property name="kinematics_offsets" value="${xacro.load_yaml('$(find motoman_gp20hl_support)' + '/config/default_kinematic_offsets.yaml')}"/>
+  <xacro:motoman_gp20hl prefix="" kinematic_offsets="${kinematics_offsets['kinematic_offsets']}"/>
 </robot>

File: motoman_gp20hl_support/urdf/gp20hl_macro.xacro (robot description, xacro)
@@ -1,5 +1,5 @@
 <?xml version="1.0" ?>
 <robot xmlns:xacro="http://ros.org/wiki/xacro">
-  <xacro:macro name="motoman_gp20hl" params="prefix">
+  <xacro:macro name="motoman_gp20hl" params="prefix kinematic_offsets">
     <xacro:include filename="$(find motoman_resources)/urdf/common_materials.xacro"/>
     <!-- link list -->
@@ -100,5 +100,5 @@
       <parent link="${prefix}base_link"/>
       <child link="${prefix}link_1_s"/>
-      <origin xyz="0 0 0.540" rpy="0 0 0" />
+      <origin xyz="${0 + kinematic_offsets['1_s']['x']} ${0 + kinematic_offsets['1_s']['y']} ${0.540 + kinematic_offsets['1_s']['z']}" rpy="${0 + kinematic_offsets['1_s']['roll']} ${0 + kinematic_offsets['1_s']['pitch']} ${0 + kinematic_offsets['1_s']['yaw']}" />
       <axis xyz="0 0 1" />
       <limit lower="${radians(-180)}" upper="${radians(180)}" effort="5516.2" velocity="${radians(180)}"/>
@@ -107,5 +107,5 @@
       <parent link="${prefix}link_1_s"/>
       <child link="${prefix}link_2_l"/>
-      <origin xyz="0.145 0 0" rpy="0 0 0" />
+      <origin xyz="${0.145 + kinematic_offsets['2_l']['x']} ${0 + kinematic_offsets['2_l']['y']} ${0 + kinematic_offsets['2_l']['z']}" rpy="${0 + kinematic_offsets['2_l']['roll']} ${0 + kinematic_offsets['2_l']['pitch']} ${0 + kinematic_offsets['2_l']['yaw']}" />
       <axis xyz="0 1 0" />
       <limit lower="${radians(-90)}" upper="${radians(135)}" effort="7060.7" velocity="${radians(180)}"/>
@@ -114,5 +114,5 @@
       <parent link="${prefix}link_2_l"/>
       <child link="${prefix}link_3_u"/>
-      <origin xyz="0 0 1.150" rpy="0 0 0" />
+      <origin xyz="${0 + kinematic_offsets['3_u']['x']} ${0 + kinematic_offsets['3_u']['y']} ${1.150 + kinematic_offsets['3_u']['z']}" rpy="${0 + kinematic_offsets['3_u']['roll']} ${0 + kinematic_offsets['3_u']['pitch']} ${0 + kinematic_offsets['3_u']['yaw']}" />
       <axis xyz="0 -1 0" />
       <limit lower="${radians(-80)}" upper="${radians(206)}" effort="3089.0" velocity="${radians(180)}"/>
@@ -121,5 +121,5 @@
       <parent link="${prefix}link_3_u"/>
       <child link="${prefix}link_4_r"/>
-      <origin xyz="1.812 0 0.250" rpy="0 0 0" />
+      <origin xyz="${1.812 + kinematic_offsets['4_r']['x']} ${0 + kinematic_offsets['4_r']['y']} ${0.250 + kinematic_offsets['4_r']['z']}" rpy="${0 + kinematic_offsets['4_r']['roll']} ${0 + kinematic_offsets['4_r']['pitch']} ${0 + kinematic_offsets['4_r']['yaw']}" />
       <axis xyz="-1 0 0" />
       <limit lower="${radians(-200)}" upper="${radians(200)}" effort="194.4" velocity="${radians(400)}"/>
@@ -128,5 +128,5 @@
       <parent link="${prefix}link_4_r"/>
       <child link="${prefix}link_5_b"/>
-      <origin xyz="0 0 0" rpy="0 0 0" />
+      <origin xyz="${0 + kinematic_offsets['5_b']['x']} ${0 + kinematic_offsets['5_b']['y']} ${0 + kinematic_offsets['5_b']['z']}" rpy="${0 + kinematic_offsets['5_b']['roll']} ${0 + kinematic_offsets['5_b']['pitch']} ${0 + kinematic_offsets['5_b']['yaw']}" />
       <axis xyz="0 -1 0" />
       <limit lower="${radians(-150)}" upper="${radians(150)}" effort="70.56" velocity="${radians(430)}"/>
@@ -135,5 +135,5 @@
       <parent link="${prefix}link_5_b"/>
       <child link="${prefix}link_6_t"/>
-      <origin xyz="0 0 0" rpy="0 0 0" />
+      <origin xyz="${0 + kinematic_offsets['6_t']['x']} ${0 + kinematic_offsets['6_t']['y']} ${0 + kinematic_offsets['6_t']['z']}" rpy="${0 + kinematic_offsets['6_t']['roll']} ${0 + kinematic_offsets['6_t']['pitch']} ${0 + kinematic_offsets['6_t']['yaw']}" />
       <axis xyz="-1 0 0" />
       <limit lower="${radians(-455)}" upper="${radians(455)}" effort="50.31" velocity="${radians(630)}"/>

File: motoman_motopos_d500_support/urdf/motopos_d500.xacro (robot description, xacro)
@@ -6,4 +6,5 @@
   </material>
   <xacro:include filename="$(find motoman_motopos_d500_support)/urdf/motopos_d500_macro.xacro" />
-  <xacro:motoman_motopos_d500 prefix=""/>
+  <xacro:property name="kinematics_offsets" value="${xacro.load_yaml('$(find motoman_motopos_d500_support)' + '/config/default_kinematic_offsets.yaml')}"/>
+  <xacro:motoman_motopos_d500 prefix="" kinematic_offsets="${kinematics_offsets['kinematic_offsets']}"/>
 </robot>

File: motoman_motopos_d500_support/urdf/motopos_d500_macro.xacro (robot description, xacro)
@@ -1,5 +1,5 @@
 <?xml version="1.0" ?>
 <robot xmlns:xacro="http://ros.org/wiki/xacro">
-  <xacro:macro name="motoman_motopos_d500" params="prefix">
+  <xacro:macro name="motoman_motopos_d500" params="prefix kinematic_offsets">
     <xacro:include filename="$(find motoman_resources)/urdf/common_materials.xacro"/>
     <!-- link list -->
@@ -48,5 +48,5 @@
       <parent link="${prefix}base_link"/>
       <child link="${prefix}link_1"/>
-      <origin xyz="0 0 0.380" rpy="0 0 0" />
+      <origin xyz="${0 + kinematic_offsets['link_1']['x']} ${0 + kinematic_offsets['link_1']['y']} ${0.380 + kinematic_offsets['link_1']['z']}" rpy="${0 + kinematic_offsets['link_1']['roll']} ${0 + kinematic_offsets['link_1']['pitch']} ${0 + kinematic_offsets['link_1']['yaw']}" />
       <axis xyz="0 -1 0" />
       <limit lower="${radians(-135)}" upper="${radians(135)}" effort="1274" velocity="${radians(80)}"/>
@@ -55,5 +55,5 @@
       <parent link="${prefix}link_1"/>
       <child link="${prefix}link_2"/>
-      <origin xyz="0 0 0" rpy="0 0 0" />
+      <origin xyz="${0 + kinematic_offsets['link_2']['x']} ${0 + kinematic_offsets['link_2']['y']} ${0 + kinematic_offsets['link_2']['z']}" rpy="${0 + kinematic_offsets['link_2']['roll']} ${0 + kinematic_offsets['link_2']['pitch']} ${0 + kinematic_offsets['link_2']['yaw']}" />
       <axis xyz="0 0 -1" />
       <limit lower="${radians(-200)}" upper="${radians(200)}" effort="392" velocity="${radians(160)}"/>

File: motoman_motopos_d500_support/urdf/motopos_d500f.xacro (robot description, xacro)
@@ -6,4 +6,5 @@
   </material>
   <xacro:include filename="$(find motoman_motopos_d500_support)/urdf/motopos_d500f_macro.xacro" />
-  <xacro:motoman_motopos_d500f prefix=""/>
+  <xacro:property name="kinematics_offsets" value="${xacro.load_yaml('$(find motoman_motopos_d500_support)' + '/config/default_kinematic_offsets.yaml')}"/>
+  <xacro:motoman_motopos_d500f prefix="" kinematic_offsets="${kinematics_offsets['kinematic_offsets']}"/>
 </robot>

File: motoman_motopos_d500_support/urdf/motopos_d500f_macro.xacro (robot description, xacro)
@@ -1,5 +1,5 @@
 <?xml version="1.0" ?>
 <robot xmlns:xacro="http://ros.org/wiki/xacro">
-  <xacro:macro name="motoman_motopos_d500f" params="prefix">
+  <xacro:macro name="motoman_motopos_d500f" params="prefix kinematic_offsets">
     <xacro:include filename="$(find motoman_resources)/urdf/common_materials.xacro"/>
     <!-- link list -->
@@ -48,5 +48,5 @@
       <parent link="${prefix}base_link"/>
       <child link="${prefix}link_1"/>
-      <origin xyz="0 0 0.380" rpy="0 0 0" />
+      <origin xyz="${0 + kinematic_offsets['link_1']['x']} ${0 + kinematic_offsets['link_1']['y']} ${0.380 + kinematic_offsets['link_1']['z']}" rpy="${0 + kinematic_offsets['link_1']['roll']} ${0 + kinematic_offsets['link_1']['pitch']} ${0 + kinematic_offsets['link_1']['yaw']}" />
       <axis xyz="0 1 0" />
       <limit lower="${radians(-135)}" upper="${radians(135)}" effort="1274" velocity="${radians(80)}"/>
@@ -55,5 +55,5 @@
       <parent link="${prefix}link_1"/>
       <child link="${prefix}link_2"/>
-      <origin xyz="0 0 0" rpy="0 0 0" />
+      <origin xyz="${0 + kinematic_offsets['link_2']['x']} ${0 + kinematic_offsets['link_2']['y']} ${0 + kinematic_offsets['link_2']['z']}" rpy="${0 + kinematic_offsets['link_2']['roll']} ${0 + kinematic_offsets['link_2']['pitch']} ${0 + kinematic_offsets['link_2']['yaw']}" />
       <axis xyz="0 0 1" />
       <limit lower="${radians(-200)}" upper="${radians(200)}" effort="392" velocity="${radians(160)}"/>

File: motoman_motopos_mh1655_support/urdf/motopos_mh1655.xacro (robot description, xacro)
@@ -2,4 +2,5 @@
 <robot name="motoman_motopos_mh1655" xmlns:xacro="http://ros.org/wiki/xacro">
   <xacro:include filename="$(find motoman_motopos_mh1655_support)/urdf/motopos_mh1655_macro.xacro" />
-  <xacro:motoman_motopos_mh1655 prefix="" use_pedestal="false"/>
+  <xacro:property name="kinematics_offsets" value="${xacro.load_yaml('$(find motoman_motopos_mh1655_support)' + '/config/default_kinematic_offsets.yaml')}"/>
+  <xacro:motoman_motopos_mh1655 prefix="" use_pedestal="false" kinematic_offsets="${kinematics_offsets['kinematic_offsets']}"/>
 </robot>

File: motoman_motopos_mh1655_support/urdf/motopos_mh1655_macro.xacro (robot description, xacro)
@@ -1,5 +1,5 @@
 <?xml version="1.0" ?>
 <robot xmlns:xacro="http://ros.org/wiki/xacro">
-  <xacro:macro name="motoman_motopos_mh1655" params="prefix use_pedestal:=false">
+  <xacro:macro name="motoman_motopos_mh1655" params="prefix use_pedestal:=false kinematic_offsets">
     <xacro:include filename="$(find motoman_resources)/urdf/common_materials.xacro"/>
     <!-- link list -->
@@ -51,5 +51,5 @@
       <parent link="${prefix}base_link"/>
       <child link="${prefix}link_1"/>
-      <origin xyz="0 0 0.305" rpy="0 0 0"/>
+      <origin xyz="${0 + kinematic_offsets['link_1']['x']} ${0 + kinematic_offsets['link_1']['y']} ${0.305 + kinematic_offsets['link_1']['z']}" rpy="${0 + kinematic_offsets['link_1']['roll']} ${0 + kinematic_offsets['link_1']['pitch']} ${0 + kinematic_offsets['link_1']['yaw']}"/>
       <axis xyz="1 0 0"/>
       <!-- NOTE: the velocity limit is a conservative conversion from the stated
