Commit message: Allow setting the kinematic offsets file as an arg to the robot xacro, defaulting to the config one

File: motoman_ar2010_support/urdf/ar2010.xacro (robot description, xacro)
@@ -2,5 +2,5 @@
 <robot name="motoman_ar2010" xmlns:xacro="http://ros.org/wiki/xacro">
   <xacro:include filename="$(find motoman_ar2010_support)/urdf/ar2010_macro.xacro" />
-  <xacro:property name="kinematics_offsets" value="${xacro.load_yaml('$(find motoman_ar2010_support)' + '/config/default_kinematic_offsets.yaml')}"/>
-  <xacro:motoman_ar2010 prefix="" kinematic_offsets="${kinematics_offsets['kinematic_offsets']}"/>
+  <xacro:arg name="kinematic_offsets_file" default="$(find motoman_ar2010_support)/config/default_kinematic_offsets.yaml"/>
+  <xacro:motoman_ar2010 prefix="" kinematic_offsets="${xacro.load_yaml('$(arg kinematic_offsets_file)')['kinematic_offsets']}"/>
 </robot>

File: motoman_gp180_support/urdf/gp180.xacro (robot description, xacro)
@@ -1,6 +1,6 @@
 <?xml version="1.0" ?>
 <robot name="motoman_gp180" xmlns:xacro="http://ros.org/wiki/xacro">
-    <xacro:include filename="$(find motoman_gp180_support)/urdf/gp180_macro.xacro" />
-  <xacro:property name="kinematics_offsets" value="${xacro.load_yaml('$(find motoman_gp180_support)' + '/config/default_kinematic_offsets.yaml')}"/>
-    <xacro:motoman_gp180 prefix="" kinematic_offsets="${kinematics_offsets['kinematic_offsets']}"/>
+  <xacro:include filename="$(find motoman_gp180_support)/urdf/gp180_macro.xacro" />
+  <xacro:arg name="kinematic_offsets_file" default="$(find motoman_gp180_support)/config/default_kinematic_offsets.yaml"/>
+  <xacro:motoman_gp180 prefix="" kinematic_offsets="${xacro.load_yaml('$(arg kinematic_offsets_file)')['kinematic_offsets']}"/>
 </robot>

File: motoman_gp20hl_support/urdf/gp20hl.xacro (robot description, xacro)
@@ -2,5 +2,5 @@
 <robot name="motoman_gp20hl" xmlns:xacro="http://ros.org/wiki/xacro">
   <xacro:include filename="$(find motoman_gp20hl_support)/urdf/gp20hl_macro.xacro" />
-  <xacro:property name="kinematics_offsets" value="${xacro.load_yaml('$(find motoman_gp20hl_support)' + '/config/default_kinematic_offsets.yaml')}"/>
-  <xacro:motoman_gp20hl prefix="" kinematic_offsets="${kinematics_offsets['kinematic_offsets']}"/>
+  <xacro:arg name="kinematic_offsets_file" default="$(find motoman_gp20hl_support)/config/default_kinematic_offsets.yaml"/>
+  <xacro:motoman_gp20hl prefix="" kinematic_offsets="${xacro.load_yaml('$(arg kinematic_offsets_file)')['kinematic_offsets']}"/>
 </robot>

File: motoman_motopos_d500_support/urdf/motopos_d500.xacro (robot description, xacro)
@@ -6,5 +6,5 @@
   </material>
   <xacro:include filename="$(find motoman_motopos_d500_support)/urdf/motopos_d500_macro.xacro" />
-  <xacro:property name="kinematics_offsets" value="${xacro.load_yaml('$(find motoman_motopos_d500_support)' + '/config/default_kinematic_offsets.yaml')}"/>
-  <xacro:motoman_motopos_d500 prefix="" kinematic_offsets="${kinematics_offsets['kinematic_offsets']}"/>
+  <xacro:arg name="kinematic_offsets_file" default="$(find motoman_motopos_d500_support)/config/default_kinematic_offsets.yaml"/>
+  <xacro:motoman_motopos_d500 prefix="" kinematic_offsets="${xacro.load_yaml('$(arg kinematic_offsets_file)')['kinematic_offsets']}"/>
 </robot>

File: motoman_motopos_d500_support/urdf/motopos_d500f.xacro (robot description, xacro)
@@ -6,5 +6,5 @@
   </material>
   <xacro:include filename="$(find motoman_motopos_d500_support)/urdf/motopos_d500f_macro.xacro" />
-  <xacro:property name="kinematics_offsets" value="${xacro.load_yaml('$(find motoman_motopos_d500_support)' + '/config/default_kinematic_offsets.yaml')}"/>
-  <xacro:motoman_motopos_d500f prefix="" kinematic_offsets="${kinematics_offsets['kinematic_offsets']}"/>
+  <xacro:arg name="kinematic_offsets_file" default="$(find motoman_motopos_d500_support)/config/default_kinematic_offsets.yaml"/>
+  <xacro:motoman_motopos_d500f prefix="" kinematic_offsets="${xacro.load_yaml('$(arg kinematic_offsets_file)')['kinematic_offsets']}"/>
 </robot>

File: motoman_motopos_mh1655_support/urdf/motopos_mh1655.xacro (robot description, xacro)
@@ -2,5 +2,5 @@
 <robot name="motoman_motopos_mh1655" xmlns:xacro="http://ros.org/wiki/xacro">
   <xacro:include filename="$(find motoman_motopos_mh1655_support)/urdf/motopos_mh1655_macro.xacro" />
-  <xacro:property name="kinematics_offsets" value="${xacro.load_yaml('$(find motoman_motopos_mh1655_support)' + '/config/default_kinematic_offsets.yaml')}"/>
-  <xacro:motoman_motopos_mh1655 prefix="" use_pedestal="false" kinematic_offsets="${kinematics_offsets['kinematic_offsets']}"/>
+  <xacro:arg name="kinematic_offsets_file" default="$(find motoman_motopos_mh1655_support)/config/default_kinematic_offsets.yaml"/>
+  <xacro:motoman_motopos_mh1655 prefix="" use_pedestal="false" kinematic_offsets="${xacro.load_yaml('$(arg kinematic_offsets_file)')['kinematic_offsets']}"/>
 </robot>
