Commit message: Port gp25 file-driven kinematics + calibration (Option A, retain .dae)
Co-authored-by: Claude <no-reply@anthropic.com>

File: motoman_gp25_support/urdf/gp25.xacro (robot description, xacro)
@@ -2,4 +2,5 @@
 <robot name="motoman_gp25" xmlns:xacro="http://ros.org/wiki/xacro">
   <xacro:include filename="$(find motoman_gp25_support)/urdf/gp25_macro.xacro" />
-  <xacro:motoman_gp25 prefix=""/>
+  <xacro:property name="kinematics" value="${xacro.load_yaml('$(find motoman_gp25_support)' + '/config/default_kinematics.yaml')}"/>
+  <xacro:motoman_gp25 prefix="" kinematics="${kinematics['kinematics']}"/>
 </robot>

File: motoman_gp25_support/urdf/gp25_macro.xacro (robot description, xacro)
@@ -1,5 +1,5 @@
 <?xml version="1.0" ?>
 <robot xmlns:xacro="http://ros.org/wiki/xacro">
-<xacro:macro name="motoman_gp25" params="prefix">
+<xacro:macro name="motoman_gp25" params="prefix kinematics">
     <xacro:include filename="$(find motoman_resources)/urdf/common_materials.xacro"/>
     <!-- link list -->
@@ -7,5 +7,5 @@
         <visual>
             <geometry>
-                <mesh filename="package://motoman_gp25_support/meshes/gp25/visual/base_link.dae"/>
+                <mesh filename="package://motoman_gp25_support/meshes/visual/base_link.stl"/>
             </geometry>
             <xacro:material_yaskawa_blue/>
@@ -13,5 +13,5 @@
         <collision>
             <geometry>
-                <mesh filename="package://motoman_gp25_support/meshes/gp25/collision/base_link.stl"/>
+                <mesh filename="package://motoman_gp25_support/meshes/collision/base_link.stl"/>
             </geometry>
         </collision>
@@ -20,5 +20,5 @@
         <visual>
             <geometry>
-                <mesh filename="package://motoman_gp25_support/meshes/gp25/visual/link_1.dae"/>
+                <mesh filename="package://motoman_gp25_support/meshes/visual/link_1_s.stl"/>
             </geometry>
             <xacro:material_yaskawa_blue/>
@@ -26,5 +26,5 @@
         <collision>
             <geometry>
-                <mesh filename="package://motoman_gp25_support/meshes/gp25/collision/link_1.stl"/>
+                <mesh filename="package://motoman_gp25_support/meshes/collision/link_1_s.stl"/>
             </geometry>
         </collision>
@@ -33,5 +33,5 @@
         <visual>
             <geometry>
-                <mesh filename="package://motoman_gp25_support/meshes/gp25/visual/link_2.dae"/>
+                <mesh filename="package://motoman_gp25_support/meshes/visual/link_2_l.stl"/>
             </geometry>
             <xacro:material_yaskawa_blue/>
@@ -39,5 +39,5 @@
         <collision>
             <geometry>
-                <mesh filename="package://motoman_gp25_support/meshes/gp25/collision/link_2.stl"/>
+                <mesh filename="package://motoman_gp25_support/meshes/collision/link_2_l.stl"/>
             </geometry>
         </collision>
@@ -46,5 +46,5 @@
         <visual>
             <geometry>
-                <mesh filename="package://motoman_gp25_support/meshes/gp25/visual/link_3.dae"/>
+                <mesh filename="package://motoman_gp25_support/meshes/visual/link_3_u.stl"/>
             </geometry>
             <xacro:material_yaskawa_blue/>
@@ -52,5 +52,5 @@
         <collision>
             <geometry>
-                <mesh filename="package://motoman_gp25_support/meshes/gp25/collision/link_3.stl"/>
+                <mesh filename="package://motoman_gp25_support/meshes/collision/link_3_u.stl"/>
             </geometry>
         </collision>
@@ -59,5 +59,5 @@
         <visual>
             <geometry>
-                <mesh filename="package://motoman_gp25_support/meshes/gp25/visual/link_4.dae"/>
+                <mesh filename="package://motoman_gp25_support/meshes/visual/link_4_r.stl"/>
             </geometry>
             <xacro:material_yaskawa_blue/>
@@ -65,5 +65,5 @@
         <collision>
             <geometry>
-                <mesh filename="package://motoman_gp25_support/meshes/gp25/collision/link_4.stl"/>
+                <mesh filename="package://motoman_gp25_support/meshes/collision/link_4_r.stl"/>
             </geometry>
         </collision>
@@ -72,5 +72,5 @@
         <visual>
             <geometry>
-                <mesh filename="package://motoman_gp25_support/meshes/gp25/visual/link_5.dae"/>
+                <mesh filename="package://motoman_gp25_support/meshes/visual/link_5_b.stl"/>
             </geometry>
             <xacro:material_yaskawa_blue/>
@@ -78,5 +78,5 @@
         <collision>
             <geometry>
-                <mesh filename="package://motoman_gp25_support/meshes/gp25/collision/link_5.stl"/>
+                <mesh filename="package://motoman_gp25_support/meshes/collision/link_5_b.stl"/>
             </geometry>
         </collision>
@@ -85,5 +85,5 @@
         <visual>
             <geometry>
-                <mesh filename="package://motoman_gp25_support/meshes/gp25/visual/link_6.dae"/>
+                <mesh filename="package://motoman_gp25_support/meshes/visual/link_6_t.stl"/>
             </geometry>
             <xacro:material_yaskawa_blue/>
@@ -91,5 +91,5 @@
         <collision>
             <geometry>
-                <mesh filename="package://motoman_gp25_support/meshes/gp25/collision/link_6.stl"/>
+                <mesh filename="package://motoman_gp25_support/meshes/collision/link_6_t.stl"/>
             </geometry>
         </collision>
@@ -100,6 +100,7 @@
         <parent link="${prefix}base_link"/>
         <child link="${prefix}link_1_s"/>
-        <origin xyz="0 0 0.505" rpy="0 0 0" />
-        <axis xyz="0 0 1" />
+        <origin xyz="${kinematics['1_s']['x']} ${kinematics['1_s']['y']} ${kinematics['1_s']['z']}"
+                rpy="${kinematics['1_s']['roll']} ${kinematics['1_s']['pitch']} ${kinematics['1_s']['yaw']}" />
+        <axis xyz="0 0 1"/>
         <limit lower="${radians(-180)}" upper="${radians(180)}" effort="3087" velocity="${radians(210)}"/>
     </joint>
@@ -107,6 +108,7 @@
         <parent link="${prefix}link_1_s"/>
         <child link="${prefix}link_2_l"/>
-        <origin xyz="0.150 0 0" rpy="0 0 0" />
-        <axis xyz="0 1 0" />
+        <origin xyz="${kinematics['2_l']['x']} ${kinematics['2_l']['y']} ${kinematics['2_l']['z']}"
+                rpy="${kinematics['2_l']['roll']} ${kinematics['2_l']['pitch']} ${kinematics['2_l']['yaw']}" />
+        <axis xyz="0 0 1"/>
         <limit lower="${radians(-105)}" upper="${radians(155)}" effort="3087" velocity="${radians(210)}"/>
     </joint>
@@ -114,6 +116,7 @@
         <parent link="${prefix}link_2_l"/>
         <child link="${prefix}link_3_u"/>
-        <origin xyz="0 0 0.760" rpy="0 0 0" />
-        <axis xyz="0 -1 0" />
+        <origin xyz="${kinematics['3_u']['x']} ${kinematics['3_u']['y']} ${kinematics['3_u']['z']}"
+                rpy="${kinematics['3_u']['roll']} ${kinematics['3_u']['pitch']} ${kinematics['3_u']['yaw']}" />
+        <axis xyz="0 0 1"/>
         <limit lower="${radians(-86)}" upper="${radians(160)}" effort="926.1" velocity="${radians(265)}"/>
     </joint>
@@ -121,6 +124,7 @@
         <parent link="${prefix}link_3_u"/>
         <child link="${prefix}link_4_r"/>
-        <origin xyz="0.795 0 0.200" rpy="0 0 0" />
-        <axis xyz="-1 0 0" />
+        <origin xyz="${kinematics['4_r']['x']} ${kinematics['4_r']['y']} ${kinematics['4_r']['z']}"
+                rpy="${kinematics['4_r']['roll']} ${kinematics['4_r']['pitch']} ${kinematics['4_r']['yaw']}" />
+        <axis xyz="0 0 1"/>
         <limit lower="${radians(-200)}" upper="${radians(200)}" effort="88.2" velocity="${radians(420)}"/>
     </joint>
@@ -128,13 +132,15 @@
         <parent link="${prefix}link_4_r"/>
         <child link="${prefix}link_5_b"/>
-        <origin xyz="0 0 0" rpy="0 0 0" />
-        <axis xyz="0 -1 0" />
-        <limit lower="${radians(-150)}" upper="${radians(150)}" effort="70.56" velocity="${radians(420)}"/>
+        <origin xyz="${kinematics['5_b']['x']} ${kinematics['5_b']['y']} ${kinematics['5_b']['z']}"
+                rpy="${kinematics['5_b']['roll']} ${kinematics['5_b']['pitch']} ${kinematics['5_b']['yaw']}" />
+        <axis xyz="0 0 1"/>
+        <limit lower="${radians(-155)}" upper="${radians(150)}" effort="70.56" velocity="${radians(420)}"/>
     </joint>
     <joint name="${prefix}joint_6_t" type="revolute">
         <parent link="${prefix}link_5_b"/>
         <child link="${prefix}link_6_t"/>
-        <origin xyz="0 0 0" rpy="0 0 0" />
-        <axis xyz="-1 0 0" />
+        <origin xyz="${kinematics['6_t']['x']} ${kinematics['6_t']['y']} ${kinematics['6_t']['z']}"
+                rpy="${kinematics['6_t']['roll']} ${kinematics['6_t']['pitch']} ${kinematics['6_t']['yaw']}" />
+        <axis xyz="0 0 1"/>
         <limit lower="${radians(-455)}" upper="${radians(455)}" effort="50.31" velocity="${radians(885)}"/>
     </joint>
@@ -143,21 +149,22 @@
     <link name="${prefix}base" />
     <joint name="${prefix}base_link-base" type="fixed">
-        <origin xyz="0 0 0.505" rpy="0 0 0"/>
+        <origin xyz="${kinematics['1_s']['x']} ${kinematics['1_s']['y']} ${kinematics['1_s']['z']}"
+                rpy="${kinematics['1_s']['roll']} ${kinematics['1_s']['pitch']} ${kinematics['1_s']['yaw']}" />
         <parent link="${prefix}base_link"/>
         <child link="${prefix}base"/>
     </joint>
-    <!-- ROS-Industrial 'flange' frame, attachment point for EEF models -->
-    <link name="${prefix}flange"/>
+    <!-- ROS-Industrial 'flange' frame: attachment point for EEF models -->
+    <link name="${prefix}flange" />
     <joint name="${prefix}joint_6_t-flange" type="fixed">
-      <origin xyz="0.100 0 0" rpy="0 0 0"/>
-      <parent link="${prefix}link_6_t"/>
-      <child link="${prefix}flange"/>
+        <origin xyz="0 0 0" rpy="0 ${pi/2.0} 0" />
+        <parent link="${prefix}link_6_t" />
+        <child link="${prefix}flange" />
     </joint>
-    <!-- ROS-Industrial 'tool0' frame, all-zeros tool frame -->
-    <link name="${prefix}tool0"/>
+    <!-- ROS-Industrial 'tool0' frame: all-zeros tool frame -->
+    <link name="${prefix}tool0" />
     <joint name="${prefix}flange-tool0" type="fixed">
-      <origin xyz="0 0 0" rpy="${radians(180)} ${radians(-90)} 0"/>
-      <parent link="${prefix}flange"/>
-      <child link="${prefix}tool0"/>
+        <origin xyz="0 0 0" rpy="${pi} ${-pi/2.0} 0" />
+        <parent link="${prefix}flange" />
+        <child link="${prefix}tool0" />
     </joint>
     </xacro:macro>

Commit message: feat: Add kinematic offsets for origin calibration gp25 (#4)
* Port gp25 file-driven kinematics + calibration

---------

Co-authored-by: Claude <no-reply@anthropic.com>
Co-authored-by: Copilot Autofix powered by AI <175728472+Copilot@users.noreply.github.com>

File: motoman_gp25_support/urdf/gp25.xacro (robot description, xacro)
@@ -2,4 +2,5 @@
 <robot name="motoman_gp25" xmlns:xacro="http://ros.org/wiki/xacro">
   <xacro:include filename="$(find motoman_gp25_support)/urdf/gp25_macro.xacro" />
-  <xacro:motoman_gp25 prefix=""/>
+  <xacro:arg name="kinematic_offsets_file" default="$(find motoman_gp25_support)/config/default_kinematic_offsets.yaml"/>
+  <xacro:motoman_gp25 prefix="" kinematic_offsets="${xacro.load_yaml('$(arg kinematic_offsets_file)')['kinematic_offsets']}"/>
 </robot>

File: motoman_gp25_support/urdf/gp25_macro.xacro (robot description, xacro)
@@ -1,5 +1,5 @@
 <?xml version="1.0" ?>
 <robot xmlns:xacro="http://ros.org/wiki/xacro">
-<xacro:macro name="motoman_gp25" params="prefix">
+<xacro:macro name="motoman_gp25" params="prefix kinematic_offsets">
     <xacro:include filename="$(find motoman_resources)/urdf/common_materials.xacro"/>
     <!-- link list -->
@@ -100,6 +100,7 @@
         <parent link="${prefix}base_link"/>
         <child link="${prefix}link_1_s"/>
-        <origin xyz="0 0 0.505" rpy="0 0 0" />
-        <axis xyz="0 0 1" />
+        <origin xyz="${0 + kinematic_offsets['1_s']['x']} ${0 + kinematic_offsets['1_s']['y']} ${0.505 + kinematic_offsets['1_s']['z']}"
+                rpy="${0 + kinematic_offsets['1_s']['roll']} ${0 + kinematic_offsets['1_s']['pitch']} ${0 + kinematic_offsets['1_s']['yaw']}" />
+        <axis xyz="0 0 1"/>
         <limit lower="${radians(-180)}" upper="${radians(180)}" effort="3087" velocity="${radians(210)}"/>
     </joint>
@@ -107,6 +108,7 @@
         <parent link="${prefix}link_1_s"/>
         <child link="${prefix}link_2_l"/>
-        <origin xyz="0.150 0 0" rpy="0 0 0" />
-        <axis xyz="0 1 0" />
+        <origin xyz="${0.150 + kinematic_offsets['2_l']['x']} ${0 + kinematic_offsets['2_l']['y']} ${0 + kinematic_offsets['2_l']['z']}"
+                rpy="${0 + kinematic_offsets['2_l']['roll']} ${0 + kinematic_offsets['2_l']['pitch']} ${0 + kinematic_offsets['2_l']['yaw']}" />
+        <axis xyz="0 1 0"/>
         <limit lower="${radians(-105)}" upper="${radians(155)}" effort="3087" velocity="${radians(210)}"/>
     </joint>
@@ -114,6 +116,7 @@
         <parent link="${prefix}link_2_l"/>
         <child link="${prefix}link_3_u"/>
-        <origin xyz="0 0 0.760" rpy="0 0 0" />
-        <axis xyz="0 -1 0" />
+        <origin xyz="${0 + kinematic_offsets['3_u']['x']} ${0 + kinematic_offsets['3_u']['y']} ${0.760 + kinematic_offsets['3_u']['z']}"
+                rpy="${0 + kinematic_offsets['3_u']['roll']} ${0 + kinematic_offsets['3_u']['pitch']} ${0 + kinematic_offsets['3_u']['yaw']}" />
+        <axis xyz="0 -1 0"/>
         <limit lower="${radians(-86)}" upper="${radians(160)}" effort="926.1" velocity="${radians(265)}"/>
     </joint>
@@ -121,6 +124,7 @@
         <parent link="${prefix}link_3_u"/>
         <child link="${prefix}link_4_r"/>
-        <origin xyz="0.795 0 0.200" rpy="0 0 0" />
-        <axis xyz="-1 0 0" />
+        <origin xyz="${0.795 + kinematic_offsets['4_r']['x']} ${0 + kinematic_offsets['4_r']['y']} ${0.200 + kinematic_offsets['4_r']['z']}"
+                rpy="${0 + kinematic_offsets['4_r']['roll']} ${0 + kinematic_offsets['4_r']['pitch']} ${0 + kinematic_offsets['4_r']['yaw']}" />
+        <axis xyz="-1 0 0"/>
         <limit lower="${radians(-200)}" upper="${radians(200)}" effort="88.2" velocity="${radians(420)}"/>
     </joint>
@@ -128,6 +132,7 @@
         <parent link="${prefix}link_4_r"/>
         <child link="${prefix}link_5_b"/>
-        <origin xyz="0 0 0" rpy="0 0 0" />
-        <axis xyz="0 -1 0" />
+        <origin xyz="${0 + kinematic_offsets['5_b']['x']} ${0 + kinematic_offsets['5_b']['y']} ${0 + kinematic_offsets['5_b']['z']}"
+                rpy="${0 + kinematic_offsets['5_b']['roll']} ${0 + kinematic_offsets['5_b']['pitch']} ${0 + kinematic_offsets['5_b']['yaw']}" />
+        <axis xyz="0 -1 0"/>
         <limit lower="${radians(-150)}" upper="${radians(150)}" effort="70.56" velocity="${radians(420)}"/>
     </joint>
@@ -135,6 +140,7 @@
         <parent link="${prefix}link_5_b"/>
         <child link="${prefix}link_6_t"/>
-        <origin xyz="0 0 0" rpy="0 0 0" />
-        <axis xyz="-1 0 0" />
+        <origin xyz="${0 + kinematic_offsets['6_t']['x']} ${0 + kinematic_offsets['6_t']['y']} ${0 + kinematic_offsets['6_t']['z']}"
+                rpy="${0 + kinematic_offsets['6_t']['roll']} ${0 + kinematic_offsets['6_t']['pitch']} ${0 + kinematic_offsets['6_t']['yaw']}" />
+        <axis xyz="-1 0 0"/>
         <limit lower="${radians(-455)}" upper="${radians(455)}" effort="50.31" velocity="${radians(885)}"/>
     </joint>
@@ -143,5 +149,6 @@
     <link name="${prefix}base" />
     <joint name="${prefix}base_link-base" type="fixed">
-        <origin xyz="0 0 0.505" rpy="0 0 0"/>
+        <origin xyz="${0 + kinematic_offsets['1_s']['x']} ${0 + kinematic_offsets['1_s']['y']} ${0.505 + kinematic_offsets['1_s']['z']}"
+                rpy="${0 + kinematic_offsets['1_s']['roll']} ${0 + kinematic_offsets['1_s']['pitch']} ${0 + kinematic_offsets['1_s']['yaw']}" />
         <parent link="${prefix}base_link"/>
         <child link="${prefix}base"/>
