Commit message: Restore previous flange and tool0 joints

File: motoman_gp25_support/urdf/gp25_macro.xacro (robot description, xacro)
@@ -154,17 +154,17 @@
         <child link="${prefix}base"/>
     </joint>
-    <!-- ROS-Industrial 'flange' frame: attachment point for EEF models -->
-    <link name="${prefix}flange" />
+    <!-- ROS-Industrial 'flange' frame, attachment point for EEF models -->
+    <link name="${prefix}flange"/>
     <joint name="${prefix}joint_6_t-flange" type="fixed">
-        <origin xyz="0 0 0" rpy="0 ${pi/2.0} 0" />
-        <parent link="${prefix}link_6_t" />
-        <child link="${prefix}flange" />
+      <origin xyz="0.100 0 0" rpy="0 0 0"/>
+      <parent link="${prefix}link_6_t"/>
+      <child link="${prefix}flange"/>
     </joint>
-    <!-- ROS-Industrial 'tool0' frame: all-zeros tool frame -->
-    <link name="${prefix}tool0" />
+    <!-- ROS-Industrial 'tool0' frame, all-zeros tool frame -->
+    <link name="${prefix}tool0"/>
     <joint name="${prefix}flange-tool0" type="fixed">
-        <origin xyz="0 0 0" rpy="${pi} ${-pi/2.0} 0" />
-        <parent link="${prefix}flange" />
-        <child link="${prefix}tool0" />
+      <origin xyz="0 0 0" rpy="${radians(180)} ${radians(-90)} 0"/>
+      <parent link="${prefix}flange"/>
+      <child link="${prefix}tool0"/>
     </joint>
     </xacro:macro>
