Commit message: Make pedestal a xacro arg
Correct the axis back to the z-axis

File: motoman_motopos_mh1655_support/urdf/motopos_mh1655.xacro (robot description, xacro)
@@ -3,4 +3,5 @@
   <xacro:include filename="$(find motoman_motopos_mh1655_support)/urdf/motopos_mh1655_macro.xacro" />
   <xacro:arg name="kinematic_offsets_file" default="$(find motoman_motopos_mh1655_support)/config/default_kinematic_offsets.yaml"/>
-  <xacro:motoman_motopos_mh1655 prefix="" use_pedestal="false" kinematic_offsets="${xacro.load_yaml('$(arg kinematic_offsets_file)')['kinematic_offsets']}"/>
+  <xacro:arg name="use_pedestal" default="false"/>
+  <xacro:motoman_motopos_mh1655 prefix="" use_pedestal="$(arg use_pedestal)" kinematic_offsets="${xacro.load_yaml('$(arg kinematic_offsets_file)')['kinematic_offsets']}"/>
 </robot>

File: motoman_motopos_mh1655_support/urdf/motopos_mh1655_macro.xacro (robot description, xacro)
@@ -62,7 +62,7 @@
       <child link="${prefix}link_1"/>
       <origin xyz="${0 + kinematic_offsets['link_1']['x']} ${0 + kinematic_offsets['link_1']['y']} ${base_link_offset + 0.305 + kinematic_offsets['link_1']['z']}"
-              rpy="${pi + kinematic_offsets['link_1']['roll']} ${-pi/2 + kinematic_offsets['link_1']['pitch']} ${0 + kinematic_offsets['link_1']['yaw']}"/>
+              rpy="${radians(90) + kinematic_offsets['link_1']['roll']} ${radians(-90) + kinematic_offsets['link_1']['pitch']} ${0 + kinematic_offsets['link_1']['yaw']}"/>
       <axis xyz="0 0 1"/>
-      <limit lower="${-2*pi}" upper="${2*pi}" effort="1274" velocity="1.3962"/>
+      <limit lower="${radians(-360)}" upper="${radians(360)}" effort="1274" velocity="${radians(65)}"/>
     </joint>
     <!-- end of joint list -->
@@ -74,5 +74,5 @@
       <child link="${prefix}base"/>
     </joint>
-    <!-- ROS-Industrial 'flange' frame: attachment point for EEF models -->
+    <!-- ROS-Industrial 'flange' frame, attachment point for EEF models -->
     <link name="${prefix}flange"/>
     <joint name="${prefix}joint_1-flange" type="fixed">
@@ -81,5 +81,5 @@
       <child link="${prefix}flange"/>
     </joint>
-    <!-- ROS-Industrial 'tool0' frame: all-zeros tool frame -->
+    <!-- ROS-Industrial 'tool0' frame, all-zeros tool frame -->
     <link name="${prefix}tool0"/>
     <joint name="${prefix}flange-tool0" type="fixed">
