Commit message: feat: More realistic/safe joint limits and MH1655 improvements (#5)
* More realistic limits for D500/D500F and GP20HL
* mh1655 axis/pedestal fix
* Improve AR2010 meshes
* Make pedestal a xacro arg

---------

Co-authored-by: Claude <no-reply@anthropic.com>

File: motoman_motopos_mh1655_support/urdf/motopos_mh1655_macro.xacro (robot description, xacro)
@@ -3,4 +3,10 @@
   <xacro:macro name="motoman_motopos_mh1655" params="prefix use_pedestal:=false kinematic_offsets">
     <xacro:include filename="$(find motoman_resources)/urdf/common_materials.xacro"/>
+    <xacro:if value="${use_pedestal}">
+      <xacro:property name="base_link_offset" value="0.695" />
+    </xacro:if>
+    <xacro:unless value="${use_pedestal}">
+      <xacro:property name="base_link_offset" value="0.0" />
+    </xacro:unless>
     <!-- link list -->
     <link name="${prefix}base_link">
@@ -9,4 +15,5 @@
           <mesh filename="package://motoman_motopos_mh1655_support/meshes/motopos_mh1655/visual/base_link.stl"/>
         </geometry>
+        <origin xyz="0 0 ${base_link_offset}" rpy="0 0 0"/>
         <xacro:material_yaskawa_blue/>
       </visual>
@@ -15,4 +22,5 @@
           <mesh filename="package://motoman_motopos_mh1655_support/meshes/motopos_mh1655/collision/base_link.stl"/>
         </geometry>
+        <origin xyz="0 0 ${base_link_offset}" rpy="0 0 0"/>
       </collision>
       <xacro:if value="${use_pedestal}">
@@ -22,4 +30,5 @@
             <mesh filename="package://motoman_motopos_mh1655_support/meshes/motopos_mh1655/visual/pedestal.stl"/>
           </geometry>
+          <origin xyz="0 0 ${base_link_offset}" rpy="0 0 0"/>
           <xacro:material_yaskawa_blue/>
         </visual>
@@ -28,4 +37,5 @@
             <mesh filename="package://motoman_motopos_mh1655_support/meshes/motopos_mh1655/collision/pedestal.stl"/>
           </geometry>
+          <origin xyz="0 0 ${base_link_offset}" rpy="0 0 0"/>
         </collision>
       </xacro:if>
@@ -51,8 +61,7 @@
       <parent link="${prefix}base_link"/>
       <child link="${prefix}link_1"/>
-      <origin xyz="${0 + kinematic_offsets['link_1']['x']} ${0 + kinematic_offsets['link_1']['y']} ${0.305 + kinematic_offsets['link_1']['z']}" rpy="${0 + kinematic_offsets['link_1']['roll']} ${0 + kinematic_offsets['link_1']['pitch']} ${0 + kinematic_offsets['link_1']['yaw']}"/>
-      <axis xyz="1 0 0"/>
-      <!-- NOTE: the velocity limit is a conservative conversion from the stated
-           limit in the manual: 10.8 rpm (in section 3.2.1) -->
+      <origin xyz="${0 + kinematic_offsets['link_1']['x']} ${0 + kinematic_offsets['link_1']['y']} ${base_link_offset + 0.305 + kinematic_offsets['link_1']['z']}"
+              rpy="${radians(90) + kinematic_offsets['link_1']['roll']} ${radians(-90) + kinematic_offsets['link_1']['pitch']} ${0 + kinematic_offsets['link_1']['yaw']}"/>
+      <axis xyz="0 0 1"/>
       <limit lower="${radians(-360)}" upper="${radians(360)}" effort="1274" velocity="${radians(65)}"/>
     </joint>
@@ -68,5 +77,5 @@
     <link name="${prefix}flange"/>
     <joint name="${prefix}joint_1-flange" type="fixed">
-      <origin xyz="0.2768 0 0" rpy="0 0 0"/>
+      <origin xyz="0 0 0.2768" rpy="0 0 0"/>
       <parent link="${prefix}link_1"/>
       <child link="${prefix}flange"/>
@@ -75,5 +84,5 @@
     <link name="${prefix}tool0"/>
     <joint name="${prefix}flange-tool0" type="fixed">
-      <origin xyz="0 0 0" rpy="${radians(180)} ${radians(-90)} 0"/>
+      <origin xyz="0 0 0" rpy="0 0 0"/>
       <parent link="${prefix}flange"/>
       <child link="${prefix}tool0"/>
