Commit message: More realistic limits for D500/D500F and GP20HL
mh1655 axis/pedestal fix

Improve AR2010 meshes

Co-authored-by: Claude <no-reply@anthropic.com>

File: motoman_gp20hl_support/urdf/gp20hl_macro.xacro (robot description, xacro)
@@ -137,5 +137,5 @@
       <origin xyz="${0 + kinematic_offsets['6_t']['x']} ${0 + kinematic_offsets['6_t']['y']} ${0 + kinematic_offsets['6_t']['z']}" rpy="${0 + kinematic_offsets['6_t']['roll']} ${0 + kinematic_offsets['6_t']['pitch']} ${0 + kinematic_offsets['6_t']['yaw']}" />
       <axis xyz="-1 0 0" />
-      <limit lower="${radians(-455)}" upper="${radians(455)}" effort="50.31" velocity="${radians(630)}"/>
+      <limit lower="${radians(-210)}" upper="${radians(210)}" effort="50.31" velocity="${radians(630)}"/>
     </joint>
     <!-- end of joint list -->

File: motoman_motopos_d500_support/urdf/motopos_d500_macro.xacro (robot description, xacro)
@@ -50,5 +50,5 @@
       <origin xyz="${0 + kinematic_offsets['link_1']['x']} ${0 + kinematic_offsets['link_1']['y']} ${0.380 + kinematic_offsets['link_1']['z']}" rpy="${0 + kinematic_offsets['link_1']['roll']} ${0 + kinematic_offsets['link_1']['pitch']} ${0 + kinematic_offsets['link_1']['yaw']}" />
       <axis xyz="0 -1 0" />
-      <limit lower="${radians(-135)}" upper="${radians(135)}" effort="1274" velocity="${radians(80)}"/>
+      <limit lower="${radians(-85.943669)}" upper="${radians(85.943669)}" effort="1274" velocity="${radians(80)}"/>
     </joint>
     <joint name="${prefix}joint_2" type="revolute">
@@ -57,5 +57,5 @@
       <origin xyz="${0 + kinematic_offsets['link_2']['x']} ${0 + kinematic_offsets['link_2']['y']} ${0 + kinematic_offsets['link_2']['z']}" rpy="${0 + kinematic_offsets['link_2']['roll']} ${0 + kinematic_offsets['link_2']['pitch']} ${0 + kinematic_offsets['link_2']['yaw']}" />
       <axis xyz="0 0 -1" />
-      <limit lower="${radians(-200)}" upper="${radians(200)}" effort="392" velocity="${radians(160)}"/>
+      <limit lower="${radians(-572.957795)}" upper="${radians(572.957795)}" effort="392" velocity="${radians(160)}"/>
     </joint>
     <!-- end of joint list -->

File: motoman_motopos_d500_support/urdf/motopos_d500f_macro.xacro (robot description, xacro)
@@ -50,5 +50,5 @@
       <origin xyz="${0 + kinematic_offsets['link_1']['x']} ${0 + kinematic_offsets['link_1']['y']} ${0.380 + kinematic_offsets['link_1']['z']}" rpy="${0 + kinematic_offsets['link_1']['roll']} ${0 + kinematic_offsets['link_1']['pitch']} ${0 + kinematic_offsets['link_1']['yaw']}" />
       <axis xyz="0 1 0" />
-      <limit lower="${radians(-135)}" upper="${radians(135)}" effort="1274" velocity="${radians(80)}"/>
+      <limit lower="${radians(-85.943669)}" upper="${radians(85.943669)}" effort="1274" velocity="${radians(80)}"/>
     </joint>
     <joint name="${prefix}joint_2" type="revolute">
@@ -57,5 +57,5 @@
       <origin xyz="${0 + kinematic_offsets['link_2']['x']} ${0 + kinematic_offsets['link_2']['y']} ${0 + kinematic_offsets['link_2']['z']}" rpy="${0 + kinematic_offsets['link_2']['roll']} ${0 + kinematic_offsets['link_2']['pitch']} ${0 + kinematic_offsets['link_2']['yaw']}" />
       <axis xyz="0 0 1" />
-      <limit lower="${radians(-200)}" upper="${radians(200)}" effort="392" velocity="${radians(160)}"/>
+      <limit lower="${radians(-572.957795)}" upper="${radians(572.957795)}" effort="392" velocity="${radians(160)}"/>
     </joint>
     <!-- end of joint list -->

File: motoman_motopos_mh1655_support/urdf/motopos_mh1655_macro.xacro (robot description, xacro)
@@ -3,4 +3,10 @@
   <xacro:macro name="motoman_motopos_mh1655" params="prefix use_pedestal:=false kinematic_offsets">
     <xacro:include filename="$(find motoman_resources)/urdf/common_materials.xacro"/>
+    <xacro:if value="${use_pedestal}">
+      <xacro:property name="base_link_offset" value="0.695" />
+    </xacro:if>
+    <xacro:unless value="${use_pedestal}">
+      <xacro:property name="base_link_offset" value="0.0" />
+    </xacro:unless>
     <!-- link list -->
     <link name="${prefix}base_link">
@@ -9,4 +15,5 @@
           <mesh filename="package://motoman_motopos_mh1655_support/meshes/motopos_mh1655/visual/base_link.stl"/>
         </geometry>
+        <origin xyz="0 0 ${base_link_offset}" rpy="0 0 0"/>
         <xacro:material_yaskawa_blue/>
       </visual>
@@ -15,4 +22,5 @@
           <mesh filename="package://motoman_motopos_mh1655_support/meshes/motopos_mh1655/collision/base_link.stl"/>
         </geometry>
+        <origin xyz="0 0 ${base_link_offset}" rpy="0 0 0"/>
       </collision>
       <xacro:if value="${use_pedestal}">
@@ -22,4 +30,5 @@
             <mesh filename="package://motoman_motopos_mh1655_support/meshes/motopos_mh1655/visual/pedestal.stl"/>
           </geometry>
+          <origin xyz="0 0 ${base_link_offset}" rpy="0 0 0"/>
           <xacro:material_yaskawa_blue/>
         </visual>
@@ -28,4 +37,5 @@
             <mesh filename="package://motoman_motopos_mh1655_support/meshes/motopos_mh1655/collision/pedestal.stl"/>
           </geometry>
+          <origin xyz="0 0 ${base_link_offset}" rpy="0 0 0"/>
         </collision>
       </xacro:if>
@@ -51,9 +61,8 @@
       <parent link="${prefix}base_link"/>
       <child link="${prefix}link_1"/>
-      <origin xyz="${0 + kinematic_offsets['link_1']['x']} ${0 + kinematic_offsets['link_1']['y']} ${0.305 + kinematic_offsets['link_1']['z']}" rpy="${0 + kinematic_offsets['link_1']['roll']} ${0 + kinematic_offsets['link_1']['pitch']} ${0 + kinematic_offsets['link_1']['yaw']}"/>
-      <axis xyz="1 0 0"/>
-      <!-- NOTE: the velocity limit is a conservative conversion from the stated
-           limit in the manual: 10.8 rpm (in section 3.2.1) -->
-      <limit lower="${radians(-360)}" upper="${radians(360)}" effort="1274" velocity="${radians(65)}"/>
+      <origin xyz="${0 + kinematic_offsets['link_1']['x']} ${0 + kinematic_offsets['link_1']['y']} ${base_link_offset + 0.305 + kinematic_offsets['link_1']['z']}"
+              rpy="${pi + kinematic_offsets['link_1']['roll']} ${-pi/2 + kinematic_offsets['link_1']['pitch']} ${0 + kinematic_offsets['link_1']['yaw']}"/>
+      <axis xyz="0 0 1"/>
+      <limit lower="${-2*pi}" upper="${2*pi}" effort="1274" velocity="1.3962"/>
     </joint>
     <!-- end of joint list -->
@@ -65,15 +74,15 @@
       <child link="${prefix}base"/>
     </joint>
-    <!-- ROS-Industrial 'flange' frame, attachment point for EEF models -->
+    <!-- ROS-Industrial 'flange' frame: attachment point for EEF models -->
     <link name="${prefix}flange"/>
     <joint name="${prefix}joint_1-flange" type="fixed">
-      <origin xyz="0.2768 0 0" rpy="0 0 0"/>
+      <origin xyz="0 0 0.2768" rpy="0 0 0"/>
       <parent link="${prefix}link_1"/>
       <child link="${prefix}flange"/>
     </joint>
-    <!-- ROS-Industrial 'tool0' frame, all-zeros tool frame -->
+    <!-- ROS-Industrial 'tool0' frame: all-zeros tool frame -->
     <link name="${prefix}tool0"/>
     <joint name="${prefix}flange-tool0" type="fixed">
-      <origin xyz="0 0 0" rpy="${radians(180)} ${radians(-90)} 0"/>
+      <origin xyz="0 0 0" rpy="0 0 0"/>
       <parent link="${prefix}flange"/>
       <child link="${prefix}tool0"/>

Commit message: fix: Restore the ROS 1 GP20HL link frames and meshes
The GP20HL macro took upstream's ROS-Industrial link frames (joint axes
z, y, -y, -x, -y, -x) while our kinematic offsets, the parts we mount on
the arm's middle links and forge's analytical IK were all written for the
ROS 1 frames (every joint about +z). Restore the ROS 1 joint origins, axes,
flange joint and STL meshes so calibrated arms come out where they did on
ROS 1. Keep the upstream joint limits.

Co-Authored-By: Claude Opus 5.5 <noreply@anthropic.com>

File: motoman_gp20hl_support/urdf/gp20hl_macro.xacro (robot description, xacro)
@@ -7,5 +7,5 @@
       <visual>
         <geometry>
-          <mesh filename="package://motoman_gp20hl_support/meshes/gp20hl/visual/base_link.dae"/>
+          <mesh filename="package://motoman_gp20hl_support/meshes/visual/base_link.stl"/>
         </geometry>
         <xacro:material_yaskawa_blue/>
@@ -13,5 +13,5 @@
       <collision>
         <geometry>
-          <mesh filename="package://motoman_gp20hl_support/meshes/gp20hl/collision/base_link.stl"/>
+          <mesh filename="package://motoman_gp20hl_support/meshes/collision/base_link.stl"/>
         </geometry>
       </collision>
@@ -20,5 +20,5 @@
       <visual>
         <geometry>
-          <mesh filename="package://motoman_gp20hl_support/meshes/gp20hl/visual/link_1.dae"/>
+          <mesh filename="package://motoman_gp20hl_support/meshes/visual/link_1_s.stl"/>
         </geometry>
         <xacro:material_yaskawa_blue/>
@@ -26,5 +26,5 @@
       <collision>
         <geometry>
-          <mesh filename="package://motoman_gp20hl_support/meshes/gp20hl/collision/link_1.stl"/>
+          <mesh filename="package://motoman_gp20hl_support/meshes/collision/link_1_s.stl"/>
         </geometry>
       </collision>
@@ -33,5 +33,5 @@
       <visual>
         <geometry>
-          <mesh filename="package://motoman_gp20hl_support/meshes/gp20hl/visual/link_2.dae"/>
+          <mesh filename="package://motoman_gp20hl_support/meshes/visual/link_2_l.stl"/>
         </geometry>
         <xacro:material_yaskawa_blue/>
@@ -39,5 +39,5 @@
       <collision>
         <geometry>
-          <mesh filename="package://motoman_gp20hl_support/meshes/gp20hl/collision/link_2.stl"/>
+          <mesh filename="package://motoman_gp20hl_support/meshes/collision/link_2_l.stl"/>
         </geometry>
       </collision>
@@ -46,5 +46,5 @@
       <visual>
         <geometry>
-          <mesh filename="package://motoman_gp20hl_support/meshes/gp20hl/visual/link_3.dae"/>
+          <mesh filename="package://motoman_gp20hl_support/meshes/visual/link_3_u.stl"/>
         </geometry>
         <xacro:material_yaskawa_blue/>
@@ -52,5 +52,5 @@
       <collision>
         <geometry>
-          <mesh filename="package://motoman_gp20hl_support/meshes/gp20hl/collision/link_3.stl"/>
+          <mesh filename="package://motoman_gp20hl_support/meshes/collision/link_3_u.stl"/>
         </geometry>
       </collision>
@@ -59,5 +59,5 @@
       <visual>
         <geometry>
-          <mesh filename="package://motoman_gp20hl_support/meshes/gp20hl/visual/link_4.dae"/>
+          <mesh filename="package://motoman_gp20hl_support/meshes/visual/link_4_r.stl"/>
         </geometry>
         <xacro:material_yaskawa_blue/>
@@ -65,5 +65,5 @@
       <collision>
         <geometry>
-          <mesh filename="package://motoman_gp20hl_support/meshes/gp20hl/collision/link_4.stl"/>
+          <mesh filename="package://motoman_gp20hl_support/meshes/collision/link_4_r.stl"/>
         </geometry>
       </collision>
@@ -72,5 +72,5 @@
       <visual>
         <geometry>
-          <mesh filename="package://motoman_gp20hl_support/meshes/gp20hl/visual/link_5.dae"/>
+          <mesh filename="package://motoman_gp20hl_support/meshes/visual/link_5_b.stl"/>
         </geometry>
         <xacro:material_yaskawa_blue/>
@@ -78,5 +78,5 @@
       <collision>
         <geometry>
-          <mesh filename="package://motoman_gp20hl_support/meshes/gp20hl/collision/link_5.stl"/>
+          <mesh filename="package://motoman_gp20hl_support/meshes/collision/link_5_b.stl"/>
         </geometry>
       </collision>
@@ -85,11 +85,11 @@
       <visual>
         <geometry>
-          <mesh filename="package://motoman_gp20hl_support/meshes/gp20hl/visual/link_6.dae"/>
+          <mesh filename="package://motoman_gp20hl_support/meshes/visual/link_6_t.stl"/>
         </geometry>
-        <xacro:material_yaskawa_silver/>
+        <xacro:material_yaskawa_blue/>
       </visual>
       <collision>
         <geometry>
-          <mesh filename="package://motoman_gp20hl_support/meshes/gp20hl/collision/link_6.stl"/>
+          <mesh filename="package://motoman_gp20hl_support/meshes/collision/link_6_t.stl"/>
         </geometry>
       </collision>
@@ -97,9 +97,11 @@
     <!-- end of link list -->
     <!-- joint list -->
+    <!-- Joints are specified such that the driver rotates the joints about the positive Z axis. -->
     <joint name="${prefix}joint_1_s" type="revolute">
       <parent link="${prefix}base_link"/>
       <child link="${prefix}link_1_s"/>
-      <origin xyz="${0 + kinematic_offsets['1_s']['x']} ${0 + kinematic_offsets['1_s']['y']} ${0.540 + kinematic_offsets['1_s']['z']}" rpy="${0 + kinematic_offsets['1_s']['roll']} ${0 + kinematic_offsets['1_s']['pitch']} ${0 + kinematic_offsets['1_s']['yaw']}" />
-      <axis xyz="0 0 1" />
+      <origin xyz="${0 + kinematic_offsets['1_s']['x']} ${0 + kinematic_offsets['1_s']['y']} ${0.540 + kinematic_offsets['1_s']['z']}"
+              rpy="${0 + kinematic_offsets['1_s']['roll']} ${0 + kinematic_offsets['1_s']['pitch']} ${0 + kinematic_offsets['1_s']['yaw']}"/>
+      <axis xyz="0 0 1"/>
       <limit lower="${radians(-180)}" upper="${radians(180)}" effort="5516.2" velocity="${radians(180)}"/>
     </joint>
@@ -107,6 +109,7 @@
       <parent link="${prefix}link_1_s"/>
       <child link="${prefix}link_2_l"/>
-      <origin xyz="${0.145 + kinematic_offsets['2_l']['x']} ${0 + kinematic_offsets['2_l']['y']} ${0 + kinematic_offsets['2_l']['z']}" rpy="${0 + kinematic_offsets['2_l']['roll']} ${0 + kinematic_offsets['2_l']['pitch']} ${0 + kinematic_offsets['2_l']['yaw']}" />
-      <axis xyz="0 1 0" />
+      <origin xyz="${0.145 + kinematic_offsets['2_l']['x']} ${0 + kinematic_offsets['2_l']['y']} ${0 + kinematic_offsets['2_l']['z']}"
+              rpy="${0 + kinematic_offsets['2_l']['roll']} ${radians(-90) + kinematic_offsets['2_l']['pitch']} ${radians(-90) + kinematic_offsets['2_l']['yaw']}"/>
+      <axis xyz="0 0 1"/>
       <limit lower="${radians(-90)}" upper="${radians(135)}" effort="7060.7" velocity="${radians(180)}"/>
     </joint>
@@ -114,6 +117,7 @@
       <parent link="${prefix}link_2_l"/>
       <child link="${prefix}link_3_u"/>
-      <origin xyz="${0 + kinematic_offsets['3_u']['x']} ${0 + kinematic_offsets['3_u']['y']} ${1.150 + kinematic_offsets['3_u']['z']}" rpy="${0 + kinematic_offsets['3_u']['roll']} ${0 + kinematic_offsets['3_u']['pitch']} ${0 + kinematic_offsets['3_u']['yaw']}" />
-      <axis xyz="0 -1 0" />
+      <origin xyz="${1.150 + kinematic_offsets['3_u']['x']} ${0 + kinematic_offsets['3_u']['y']} ${0 + kinematic_offsets['3_u']['z']}"
+              rpy="${radians(180) + kinematic_offsets['3_u']['roll']} ${0 + kinematic_offsets['3_u']['pitch']} ${0 + kinematic_offsets['3_u']['yaw']}"/>
+      <axis xyz="0 0 1"/>
       <limit lower="${radians(-80)}" upper="${radians(206)}" effort="3089.0" velocity="${radians(180)}"/>
     </joint>
@@ -121,6 +125,7 @@
       <parent link="${prefix}link_3_u"/>
       <child link="${prefix}link_4_r"/>
-      <origin xyz="${1.812 + kinematic_offsets['4_r']['x']} ${0 + kinematic_offsets['4_r']['y']} ${0.250 + kinematic_offsets['4_r']['z']}" rpy="${0 + kinematic_offsets['4_r']['roll']} ${0 + kinematic_offsets['4_r']['pitch']} ${0 + kinematic_offsets['4_r']['yaw']}" />
-      <axis xyz="-1 0 0" />
+      <origin xyz="${0.250 + kinematic_offsets['4_r']['x']} ${-1.812 + kinematic_offsets['4_r']['y']} ${0 + kinematic_offsets['4_r']['z']}"
+              rpy="${radians(-90) + kinematic_offsets['4_r']['roll']} ${0 + kinematic_offsets['4_r']['pitch']} ${0 + kinematic_offsets['4_r']['yaw']}"/>
+      <axis xyz="0 0 1"/>
       <limit lower="${radians(-200)}" upper="${radians(200)}" effort="194.4" velocity="${radians(400)}"/>
     </joint>
@@ -128,6 +133,7 @@
       <parent link="${prefix}link_4_r"/>
       <child link="${prefix}link_5_b"/>
-      <origin xyz="${0 + kinematic_offsets['5_b']['x']} ${0 + kinematic_offsets['5_b']['y']} ${0 + kinematic_offsets['5_b']['z']}" rpy="${0 + kinematic_offsets['5_b']['roll']} ${0 + kinematic_offsets['5_b']['pitch']} ${0 + kinematic_offsets['5_b']['yaw']}" />
-      <axis xyz="0 -1 0" />
+      <origin xyz="${0 + kinematic_offsets['5_b']['x']} ${0 + kinematic_offsets['5_b']['y']} ${0 + kinematic_offsets['5_b']['z']}"
+              rpy="${radians(90) + kinematic_offsets['5_b']['roll']} ${0 + kinematic_offsets['5_b']['pitch']} ${0 + kinematic_offsets['5_b']['yaw']}"/>
+      <axis xyz="0 0 1"/>
       <limit lower="${radians(-150)}" upper="${radians(150)}" effort="70.56" velocity="${radians(430)}"/>
     </joint>
@@ -135,11 +141,12 @@
       <parent link="${prefix}link_5_b"/>
       <child link="${prefix}link_6_t"/>
-      <origin xyz="${0 + kinematic_offsets['6_t']['x']} ${0 + kinematic_offsets['6_t']['y']} ${0 + kinematic_offsets['6_t']['z']}" rpy="${0 + kinematic_offsets['6_t']['roll']} ${0 + kinematic_offsets['6_t']['pitch']} ${0 + kinematic_offsets['6_t']['yaw']}" />
-      <axis xyz="-1 0 0" />
+      <origin xyz="${0 + kinematic_offsets['6_t']['x']} ${-0.1 + kinematic_offsets['6_t']['y']} ${0 + kinematic_offsets['6_t']['z']}"
+              rpy="${radians(-90) + kinematic_offsets['6_t']['roll']} ${0 + kinematic_offsets['6_t']['pitch']} ${0 + kinematic_offsets['6_t']['yaw']}"/>
+      <axis xyz="0 0 1"/>
       <limit lower="${radians(-210)}" upper="${radians(210)}" effort="50.31" velocity="${radians(630)}"/>
     </joint>
     <!-- end of joint list -->
     <!-- ROS base_link to Robot Manufacturer World Coordinates transform -->
-    <link name="${prefix}base" />
+    <link name="${prefix}base"/>
     <joint name="${prefix}base_link-base" type="fixed">
       <origin xyz="0 0 0.540" rpy="0 0 0"/>
@@ -147,15 +154,15 @@
       <child link="${prefix}base"/>
     </joint>
-    <!-- ROS-Industrial 'flange' frame, attachment point for EEF models -->
+    <!-- ROS-Industrial 'flange' frame: attachment point for EEF models -->
     <link name="${prefix}flange"/>
     <joint name="${prefix}joint_6_t-flange" type="fixed">
-      <origin xyz="0.100 0 0" rpy="0 0 0"/>
+      <origin xyz="0 0 0" rpy="0 ${pi/2} 0"/>
       <parent link="${prefix}link_6_t"/>
       <child link="${prefix}flange"/>
     </joint>
-    <!-- ROS-Industrial 'tool0' frame, all-zeros tool frame -->
+    <!-- ROS-Industrial 'tool0' frame: all-zeros tool frame -->
     <link name="${prefix}tool0"/>
     <joint name="${prefix}flange-tool0" type="fixed">
-      <origin xyz="0 0 0" rpy="${radians(180)} ${radians(-90)} 0"/>
+      <origin xyz="0 0 0" rpy="${pi} ${-pi/2.0} 0"/>
       <parent link="${prefix}flange"/>
       <child link="${prefix}tool0"/>

Commit message: refactor: Keep the GP20HL meshes at upstream's paths
Move the restored ROS 1 meshes to meshes/gp20hl/{collision,visual}/link_N.stl,
the same way the AR2010 and GP180 meshes were carried over. The files are
unchanged.

Co-Authored-By: Claude Opus 5.5 <noreply@anthropic.com>

File: motoman_gp20hl_support/urdf/gp20hl_macro.xacro (robot description, xacro)
@@ -7,5 +7,5 @@
       <visual>
         <geometry>
-          <mesh filename="package://motoman_gp20hl_support/meshes/visual/base_link.stl"/>
+          <mesh filename="package://motoman_gp20hl_support/meshes/gp20hl/visual/base_link.stl"/>
         </geometry>
         <xacro:material_yaskawa_blue/>
@@ -13,5 +13,5 @@
       <collision>
         <geometry>
-          <mesh filename="package://motoman_gp20hl_support/meshes/collision/base_link.stl"/>
+          <mesh filename="package://motoman_gp20hl_support/meshes/gp20hl/collision/base_link.stl"/>
         </geometry>
       </collision>
@@ -20,5 +20,5 @@
       <visual>
         <geometry>
-          <mesh filename="package://motoman_gp20hl_support/meshes/visual/link_1_s.stl"/>
+          <mesh filename="package://motoman_gp20hl_support/meshes/gp20hl/visual/link_1.stl"/>
         </geometry>
         <xacro:material_yaskawa_blue/>
@@ -26,5 +26,5 @@
       <collision>
         <geometry>
-          <mesh filename="package://motoman_gp20hl_support/meshes/collision/link_1_s.stl"/>
+          <mesh filename="package://motoman_gp20hl_support/meshes/gp20hl/collision/link_1.stl"/>
         </geometry>
       </collision>
@@ -33,5 +33,5 @@
       <visual>
         <geometry>
-          <mesh filename="package://motoman_gp20hl_support/meshes/visual/link_2_l.stl"/>
+          <mesh filename="package://motoman_gp20hl_support/meshes/gp20hl/visual/link_2.stl"/>
         </geometry>
         <xacro:material_yaskawa_blue/>
@@ -39,5 +39,5 @@
       <collision>
         <geometry>
-          <mesh filename="package://motoman_gp20hl_support/meshes/collision/link_2_l.stl"/>
+          <mesh filename="package://motoman_gp20hl_support/meshes/gp20hl/collision/link_2.stl"/>
         </geometry>
       </collision>
@@ -46,5 +46,5 @@
       <visual>
         <geometry>
-          <mesh filename="package://motoman_gp20hl_support/meshes/visual/link_3_u.stl"/>
+          <mesh filename="package://motoman_gp20hl_support/meshes/gp20hl/visual/link_3.stl"/>
         </geometry>
         <xacro:material_yaskawa_blue/>
@@ -52,5 +52,5 @@
       <collision>
         <geometry>
-          <mesh filename="package://motoman_gp20hl_support/meshes/collision/link_3_u.stl"/>
+          <mesh filename="package://motoman_gp20hl_support/meshes/gp20hl/collision/link_3.stl"/>
         </geometry>
       </collision>
@@ -59,5 +59,5 @@
       <visual>
         <geometry>
-          <mesh filename="package://motoman_gp20hl_support/meshes/visual/link_4_r.stl"/>
+          <mesh filename="package://motoman_gp20hl_support/meshes/gp20hl/visual/link_4.stl"/>
         </geometry>
         <xacro:material_yaskawa_blue/>
@@ -65,5 +65,5 @@
       <collision>
         <geometry>
-          <mesh filename="package://motoman_gp20hl_support/meshes/collision/link_4_r.stl"/>
+          <mesh filename="package://motoman_gp20hl_support/meshes/gp20hl/collision/link_4.stl"/>
         </geometry>
       </collision>
@@ -72,5 +72,5 @@
       <visual>
         <geometry>
-          <mesh filename="package://motoman_gp20hl_support/meshes/visual/link_5_b.stl"/>
+          <mesh filename="package://motoman_gp20hl_support/meshes/gp20hl/visual/link_5.stl"/>
         </geometry>
         <xacro:material_yaskawa_blue/>
@@ -78,5 +78,5 @@
       <collision>
         <geometry>
-          <mesh filename="package://motoman_gp20hl_support/meshes/collision/link_5_b.stl"/>
+          <mesh filename="package://motoman_gp20hl_support/meshes/gp20hl/collision/link_5.stl"/>
         </geometry>
       </collision>
@@ -85,5 +85,5 @@
       <visual>
         <geometry>
-          <mesh filename="package://motoman_gp20hl_support/meshes/visual/link_6_t.stl"/>
+          <mesh filename="package://motoman_gp20hl_support/meshes/gp20hl/visual/link_6.stl"/>
         </geometry>
         <xacro:material_yaskawa_blue/>
@@ -91,5 +91,5 @@
       <collision>
         <geometry>
-          <mesh filename="package://motoman_gp20hl_support/meshes/collision/link_6_t.stl"/>
+          <mesh filename="package://motoman_gp20hl_support/meshes/gp20hl/collision/link_6.stl"/>
         </geometry>
       </collision>
