Commit message: fix: Restore original GP20HL link frames and meshes (#6)
* fix: Restore the ROS 1 GP20HL link frames and meshes

The GP20HL macro took upstream's ROS-Industrial link frames (joint axes
z, y, -y, -x, -y, -x) while our kinematic offsets, the parts we mount on
the arm's middle links and forge's analytical IK were all written for the
ROS 1 frames (every joint about +z). Restore the ROS 1 joint origins, axes,
flange joint and STL meshes so calibrated arms come out where they did on
ROS 1. Keep the upstream joint limits.

Co-Authored-By: Claude Opus 5.5 <noreply@anthropic.com>

* refactor: Keep the GP20HL meshes at upstream's paths

Move the restored ROS 1 meshes to meshes/gp20hl/{collision,visual}/link_N.stl,
the same way the AR2010 and GP180 meshes were carried over. The files are
unchanged.

Co-Authored-By: Claude Opus 5.5 <noreply@anthropic.com>

---------

Co-authored-by: Claude Opus 5.5 <noreply@anthropic.com>

File: motoman_gp20hl_support/urdf/gp20hl_macro.xacro (robot description, xacro)
@@ -7,5 +7,5 @@
       <visual>
         <geometry>
-          <mesh filename="package://motoman_gp20hl_support/meshes/gp20hl/visual/base_link.dae"/>
+          <mesh filename="package://motoman_gp20hl_support/meshes/gp20hl/visual/base_link.stl"/>
         </geometry>
         <xacro:material_yaskawa_blue/>
@@ -20,5 +20,5 @@
       <visual>
         <geometry>
-          <mesh filename="package://motoman_gp20hl_support/meshes/gp20hl/visual/link_1.dae"/>
+          <mesh filename="package://motoman_gp20hl_support/meshes/gp20hl/visual/link_1.stl"/>
         </geometry>
         <xacro:material_yaskawa_blue/>
@@ -33,5 +33,5 @@
       <visual>
         <geometry>
-          <mesh filename="package://motoman_gp20hl_support/meshes/gp20hl/visual/link_2.dae"/>
+          <mesh filename="package://motoman_gp20hl_support/meshes/gp20hl/visual/link_2.stl"/>
         </geometry>
         <xacro:material_yaskawa_blue/>
@@ -46,5 +46,5 @@
       <visual>
         <geometry>
-          <mesh filename="package://motoman_gp20hl_support/meshes/gp20hl/visual/link_3.dae"/>
+          <mesh filename="package://motoman_gp20hl_support/meshes/gp20hl/visual/link_3.stl"/>
         </geometry>
         <xacro:material_yaskawa_blue/>
@@ -59,5 +59,5 @@
       <visual>
         <geometry>
-          <mesh filename="package://motoman_gp20hl_support/meshes/gp20hl/visual/link_4.dae"/>
+          <mesh filename="package://motoman_gp20hl_support/meshes/gp20hl/visual/link_4.stl"/>
         </geometry>
         <xacro:material_yaskawa_blue/>
@@ -72,5 +72,5 @@
       <visual>
         <geometry>
-          <mesh filename="package://motoman_gp20hl_support/meshes/gp20hl/visual/link_5.dae"/>
+          <mesh filename="package://motoman_gp20hl_support/meshes/gp20hl/visual/link_5.stl"/>
         </geometry>
         <xacro:material_yaskawa_blue/>
@@ -85,7 +85,7 @@
       <visual>
         <geometry>
-          <mesh filename="package://motoman_gp20hl_support/meshes/gp20hl/visual/link_6.dae"/>
+          <mesh filename="package://motoman_gp20hl_support/meshes/gp20hl/visual/link_6.stl"/>
         </geometry>
-        <xacro:material_yaskawa_silver/>
+        <xacro:material_yaskawa_blue/>
       </visual>
       <collision>
@@ -97,9 +97,11 @@
     <!-- end of link list -->
     <!-- joint list -->
+    <!-- Joints are specified such that the driver rotates the joints about the positive Z axis. -->
     <joint name="${prefix}joint_1_s" type="revolute">
       <parent link="${prefix}base_link"/>
       <child link="${prefix}link_1_s"/>
-      <origin xyz="${0 + kinematic_offsets['1_s']['x']} ${0 + kinematic_offsets['1_s']['y']} ${0.540 + kinematic_offsets['1_s']['z']}" rpy="${0 + kinematic_offsets['1_s']['roll']} ${0 + kinematic_offsets['1_s']['pitch']} ${0 + kinematic_offsets['1_s']['yaw']}" />
-      <axis xyz="0 0 1" />
+      <origin xyz="${0 + kinematic_offsets['1_s']['x']} ${0 + kinematic_offsets['1_s']['y']} ${0.540 + kinematic_offsets['1_s']['z']}"
+              rpy="${0 + kinematic_offsets['1_s']['roll']} ${0 + kinematic_offsets['1_s']['pitch']} ${0 + kinematic_offsets['1_s']['yaw']}"/>
+      <axis xyz="0 0 1"/>
       <limit lower="${radians(-180)}" upper="${radians(180)}" effort="5516.2" velocity="${radians(180)}"/>
     </joint>
@@ -107,6 +109,7 @@
       <parent link="${prefix}link_1_s"/>
       <child link="${prefix}link_2_l"/>
-      <origin xyz="${0.145 + kinematic_offsets['2_l']['x']} ${0 + kinematic_offsets['2_l']['y']} ${0 + kinematic_offsets['2_l']['z']}" rpy="${0 + kinematic_offsets['2_l']['roll']} ${0 + kinematic_offsets['2_l']['pitch']} ${0 + kinematic_offsets['2_l']['yaw']}" />
-      <axis xyz="0 1 0" />
+      <origin xyz="${0.145 + kinematic_offsets['2_l']['x']} ${0 + kinematic_offsets['2_l']['y']} ${0 + kinematic_offsets['2_l']['z']}"
+              rpy="${0 + kinematic_offsets['2_l']['roll']} ${radians(-90) + kinematic_offsets['2_l']['pitch']} ${radians(-90) + kinematic_offsets['2_l']['yaw']}"/>
+      <axis xyz="0 0 1"/>
       <limit lower="${radians(-90)}" upper="${radians(135)}" effort="7060.7" velocity="${radians(180)}"/>
     </joint>
@@ -114,6 +117,7 @@
       <parent link="${prefix}link_2_l"/>
       <child link="${prefix}link_3_u"/>
-      <origin xyz="${0 + kinematic_offsets['3_u']['x']} ${0 + kinematic_offsets['3_u']['y']} ${1.150 + kinematic_offsets['3_u']['z']}" rpy="${0 + kinematic_offsets['3_u']['roll']} ${0 + kinematic_offsets['3_u']['pitch']} ${0 + kinematic_offsets['3_u']['yaw']}" />
-      <axis xyz="0 -1 0" />
+      <origin xyz="${1.150 + kinematic_offsets['3_u']['x']} ${0 + kinematic_offsets['3_u']['y']} ${0 + kinematic_offsets['3_u']['z']}"
+              rpy="${radians(180) + kinematic_offsets['3_u']['roll']} ${0 + kinematic_offsets['3_u']['pitch']} ${0 + kinematic_offsets['3_u']['yaw']}"/>
+      <axis xyz="0 0 1"/>
       <limit lower="${radians(-80)}" upper="${radians(206)}" effort="3089.0" velocity="${radians(180)}"/>
     </joint>
@@ -121,6 +125,7 @@
       <parent link="${prefix}link_3_u"/>
       <child link="${prefix}link_4_r"/>
-      <origin xyz="${1.812 + kinematic_offsets['4_r']['x']} ${0 + kinematic_offsets['4_r']['y']} ${0.250 + kinematic_offsets['4_r']['z']}" rpy="${0 + kinematic_offsets['4_r']['roll']} ${0 + kinematic_offsets['4_r']['pitch']} ${0 + kinematic_offsets['4_r']['yaw']}" />
-      <axis xyz="-1 0 0" />
+      <origin xyz="${0.250 + kinematic_offsets['4_r']['x']} ${-1.812 + kinematic_offsets['4_r']['y']} ${0 + kinematic_offsets['4_r']['z']}"
+              rpy="${radians(-90) + kinematic_offsets['4_r']['roll']} ${0 + kinematic_offsets['4_r']['pitch']} ${0 + kinematic_offsets['4_r']['yaw']}"/>
+      <axis xyz="0 0 1"/>
       <limit lower="${radians(-200)}" upper="${radians(200)}" effort="194.4" velocity="${radians(400)}"/>
     </joint>
@@ -128,6 +133,7 @@
       <parent link="${prefix}link_4_r"/>
       <child link="${prefix}link_5_b"/>
-      <origin xyz="${0 + kinematic_offsets['5_b']['x']} ${0 + kinematic_offsets['5_b']['y']} ${0 + kinematic_offsets['5_b']['z']}" rpy="${0 + kinematic_offsets['5_b']['roll']} ${0 + kinematic_offsets['5_b']['pitch']} ${0 + kinematic_offsets['5_b']['yaw']}" />
-      <axis xyz="0 -1 0" />
+      <origin xyz="${0 + kinematic_offsets['5_b']['x']} ${0 + kinematic_offsets['5_b']['y']} ${0 + kinematic_offsets['5_b']['z']}"
+              rpy="${radians(90) + kinematic_offsets['5_b']['roll']} ${0 + kinematic_offsets['5_b']['pitch']} ${0 + kinematic_offsets['5_b']['yaw']}"/>
+      <axis xyz="0 0 1"/>
       <limit lower="${radians(-150)}" upper="${radians(150)}" effort="70.56" velocity="${radians(430)}"/>
     </joint>
@@ -135,11 +141,12 @@
       <parent link="${prefix}link_5_b"/>
       <child link="${prefix}link_6_t"/>
-      <origin xyz="${0 + kinematic_offsets['6_t']['x']} ${0 + kinematic_offsets['6_t']['y']} ${0 + kinematic_offsets['6_t']['z']}" rpy="${0 + kinematic_offsets['6_t']['roll']} ${0 + kinematic_offsets['6_t']['pitch']} ${0 + kinematic_offsets['6_t']['yaw']}" />
-      <axis xyz="-1 0 0" />
+      <origin xyz="${0 + kinematic_offsets['6_t']['x']} ${-0.1 + kinematic_offsets['6_t']['y']} ${0 + kinematic_offsets['6_t']['z']}"
+              rpy="${radians(-90) + kinematic_offsets['6_t']['roll']} ${0 + kinematic_offsets['6_t']['pitch']} ${0 + kinematic_offsets['6_t']['yaw']}"/>
+      <axis xyz="0 0 1"/>
       <limit lower="${radians(-210)}" upper="${radians(210)}" effort="50.31" velocity="${radians(630)}"/>
     </joint>
     <!-- end of joint list -->
     <!-- ROS base_link to Robot Manufacturer World Coordinates transform -->
-    <link name="${prefix}base" />
+    <link name="${prefix}base"/>
     <joint name="${prefix}base_link-base" type="fixed">
       <origin xyz="0 0 0.540" rpy="0 0 0"/>
@@ -147,15 +154,15 @@
       <child link="${prefix}base"/>
     </joint>
-    <!-- ROS-Industrial 'flange' frame, attachment point for EEF models -->
+    <!-- ROS-Industrial 'flange' frame: attachment point for EEF models -->
     <link name="${prefix}flange"/>
     <joint name="${prefix}joint_6_t-flange" type="fixed">
-      <origin xyz="0.100 0 0" rpy="0 0 0"/>
+      <origin xyz="0 0 0" rpy="0 ${pi/2} 0"/>
       <parent link="${prefix}link_6_t"/>
       <child link="${prefix}flange"/>
     </joint>
-    <!-- ROS-Industrial 'tool0' frame, all-zeros tool frame -->
+    <!-- ROS-Industrial 'tool0' frame: all-zeros tool frame -->
     <link name="${prefix}tool0"/>
     <joint name="${prefix}flange-tool0" type="fixed">
-      <origin xyz="0 0 0" rpy="${radians(180)} ${radians(-90)} 0"/>
+      <origin xyz="0 0 0" rpy="${pi} ${-pi/2.0} 0"/>
       <parent link="${prefix}flange"/>
       <child link="${prefix}tool0"/>
